Commit message: creating launch to spawn in world

File: src/clyde_description/src/urdf/clyde_simple.xacro (robot description, xacro)
@@ -11,5 +11,5 @@
   </inertial>
 </xacro:macro>
-<xacro:property name="camera_link" value="0.05" />
+<xacro:property name="camera_link" value="0.01" />
 <link name="base_link">
   <inertial>
@@ -21,5 +21,5 @@
     <origin xyz="0 0 0" rpy="0 0 0"/>
     <geometry>
-      <mesh filename="package://clyde_description/src/meshes/base_link.stl" scale="0.001 0.001 0.001"/>
+      <mesh filename="file://$(find clyde_description)/src/models/clyde_model/meshes/base_link.stl" scale="0.001 0.001 0.001"/>
     </geometry>
     <material name="silver"/>
@@ -28,5 +28,5 @@
     <origin xyz="0 0 0" rpy="0 0 0"/>
     <geometry>
-      <mesh filename="package://clyde_description/src/meshes/base_link.stl" scale="0.001 0.001 0.001"/>
+      <mesh filename="file://$(find clyde_description)/src/models/clyde_model/meshes/base_link.stl" scale="0.001 0.001 0.001"/>
     </geometry>
   </collision>
@@ -55,5 +55,5 @@
 <joint name="camera_joint" type="fixed">
   <axis xyz="0 1 0" />
-  <origin xyz="${camera_link} 0 0" rpy="-0.32814212668464987 0.10093359552132034 -0.5922309969483743"/>
+  <origin xyz="${camera_link} 0.020 0.015" rpy="-0.32814212668464987 0.10093359552132034 -0.5922309969483743"/>
   <parent link="head__1"/>
   <child link="camera_link"/>
@@ -68,5 +68,5 @@
     <origin xyz="-0.061733 0.028 -0.025792" rpy="0 0 0"/>
     <geometry>
-      <mesh filename="package://clyde_description/src/meshes/front__1.stl" scale="0.001 0.001 0.001"/>
+      <mesh filename="file://$(find clyde_description)/src/models/clyde_model/meshes/front__1.stl" scale="0.001 0.001 0.001"/>
     </geometry>
     <material name="silver"/>
@@ -75,5 +75,5 @@
     <origin xyz="-0.061733 0.028 -0.025792" rpy="0 0 0"/>
     <geometry>
-      <mesh filename="package://clyde_description/src/meshes/front__1.stl" scale="0.001 0.001 0.001"/>
+      <mesh filename="file://$(find clyde_description)/src/models/clyde_model/meshes/front__1.stl" scale="0.001 0.001 0.001"/>
     </geometry>
   </collision>
@@ -88,5 +88,5 @@
     <origin xyz="0.061733 -0.028 -0.025792" rpy="0 0 0"/>
     <geometry>
-      <mesh filename="package://clyde_description/src/meshes/rear__1.stl" scale="0.001 0.001 0.001"/>
+      <mesh filename="file://$(find clyde_description)/src/models/clyde_model/meshes/rear__1.stl" scale="0.001 0.001 0.001"/>
     </geometry>
     <material name="silver"/>
@@ -95,5 +95,5 @@
     <origin xyz="0.061733 -0.028 -0.025792" rpy="0 0 0"/>
     <geometry>
-      <mesh filename="package://clyde_description/src/meshes/rear__1.stl" scale="0.001 0.001 0.001"/>
+      <mesh filename="file://$(find clyde_description)/src/models/clyde_model/meshes/rear__1.stl" scale="0.001 0.001 0.001"/>
     </geometry>
   </collision>
@@ -108,5 +108,5 @@
     <origin xyz="-0.059645 0.036 -0.017875" rpy="0 0 0"/>
     <geometry>
-      <mesh filename="package://clyde_description/src/meshes/servo_rfs_1.stl" scale="0.001 0.001 0.001"/>
+      <mesh filename="file://$(find clyde_description)/src/models/clyde_model/meshes/servo_rfs_1.stl" scale="0.001 0.001 0.001"/>
     </geometry>
     <material name="silver"/>
@@ -115,5 +115,5 @@
     <origin xyz="-0.059645 0.036 -0.017875" rpy="0 0 0"/>
     <geometry>
-      <mesh filename="package://clyde_description/src/meshes/servo_rfs_1.stl" scale="0.001 0.001 0.001"/>
+      <mesh filename="file://$(find clyde_description)/src/models/clyde_model/meshes/servo_rfs_1.stl" scale="0.001 0.001 0.001"/>
     </geometry>
   </collision>
@@ -128,5 +128,5 @@
     <origin xyz="0.059645 0.036 -0.017875" rpy="0 0 0"/>
     <geometry>
-      <mesh filename="package://clyde_description/src/meshes/servo_rrs__1.stl" scale="0.001 0.001 0.001"/>
+      <mesh filename="file://$(find clyde_description)/src/models/clyde_model/meshes/servo_rrs__1.stl" scale="0.001 0.001 0.001"/>
     </geometry>
     <material name="silver"/>
@@ -135,5 +135,5 @@
     <origin xyz="0.059645 0.036 -0.017875" rpy="0 0 0"/>
     <geometry>
-      <mesh filename="package://clyde_description/src/meshes/servo_rrs__1.stl" scale="0.001 0.001 0.001"/>
+      <mesh filename="file://$(find clyde_description)/src/models/clyde_model/meshes/servo_rrs__1.stl" scale="0.001 0.001 0.001"/>
     </geometry>
   </collision>
@@ -148,5 +148,5 @@
     <origin xyz="-0.044904 -0.0 -0.031351" rpy="0 0 0"/>
     <geometry>
-      <mesh filename="package://clyde_description/src/meshes/c_neck__1.stl" scale="0.001 0.001 0.001"/>
+      <mesh filename="file://$(find clyde_description)/src/models/clyde_model/meshes/c_neck__1.stl" scale="0.001 0.001 0.001"/>
     </geometry>
     <material name="silver"/>
@@ -155,5 +155,5 @@
     <origin xyz="-0.044904 -0.0 -0.031351" rpy="0 0 0"/>
     <geometry>
-      <mesh filename="package://clyde_description/src/meshes/c_neck__1.stl" scale="0.001 0.001 0.001"/>
+      <mesh filename="file://$(find clyde_description)/src/models/clyde_model/meshes/c_neck__1.stl" scale="0.001 0.001 0.001"/>
     </geometry>
   </collision>
@@ -168,5 +168,5 @@
     <origin xyz="-0.055711 0.017155 -0.060327" rpy="0 0 0"/>
     <geometry>
-      <mesh filename="package://clyde_description/src/meshes/head__1.stl" scale="0.001 0.001 0.001"/>
+      <mesh filename="file://$(find clyde_description)/src/models/clyde_model/meshes/head__1.stl" scale="0.001 0.001 0.001"/>
     </geometry>
     <material name="silver"/>
@@ -175,5 +175,5 @@
     <origin xyz="-0.055711 0.017155 -0.060327" rpy="0 0 0"/>
     <geometry>
-      <mesh filename="package://clyde_description/src/meshes/head__1.stl" scale="0.001 0.001 0.001"/>
+      <mesh filename="file://$(find clyde_description)/src/models/clyde_model/meshes/head__1.stl" scale="0.001 0.001 0.001"/>
     </geometry>
   </collision>
@@ -188,5 +188,5 @@
     <origin xyz="-0.06445 0.012925 -0.034027" rpy="0 0 0"/>
     <geometry>
-      <mesh filename="package://clyde_description/src/meshes/jaw_1.stl" scale="0.001 0.001 0.001"/>
+      <mesh filename="file://$(find clyde_description)/src/models/clyde_model/meshes/jaw_1.stl" scale="0.001 0.001 0.001"/>
     </geometry>
     <material name="silver"/>
@@ -195,5 +195,5 @@
     <origin xyz="-0.06445 0.012925 -0.034027" rpy="0 0 0"/>
     <geometry>
-      <mesh filename="package://clyde_description/src/meshes/jaw_1.stl" scale="0.001 0.001 0.001"/>
+      <mesh filename="file://$(find clyde_description)/src/models/clyde_model/meshes/jaw_1.stl" scale="0.001 0.001 0.001"/>
     </geometry>
   </collision>
@@ -208,5 +208,5 @@
     <origin xyz="-0.038977 0.050355 -0.018377" rpy="0 0 0"/>
     <geometry>
-      <mesh filename="package://clyde_description/src/meshes/tho_rf__1.stl" scale="0.001 0.001 0.001"/>
+      <mesh filename="file://$(find clyde_description)/src/models/clyde_model/meshes/tho_rf__1.stl" scale="0.001 0.001 0.001"/>
     </geometry>
     <material name="silver"/>
@@ -215,5 +215,5 @@
     <origin xyz="-0.038977 0.050355 -0.018377" rpy="0 0 0"/>
     <geometry>
-      <mesh filename="package://clyde_description/src/meshes/tho_rf__1.stl" scale="0.001 0.001 0.001"/>
+      <mesh filename="file://$(find clyde_description)/src/models/clyde_model/meshes/tho_rf__1.stl" scale="0.001 0.001 0.001"/>
     </geometry>
   </collision>
@@ -228,5 +228,5 @@
     <origin xyz="-0.047554 -0.0 -0.035941" rpy="0 0 0"/>
     <geometry>
-      <mesh filename="package://clyde_description/src/meshes/servo_neck__1.stl" scale="0.001 0.001 0.001"/>
+      <mesh filename="file://$(find clyde_description)/src/models/clyde_model/meshes/servo_neck__1.stl" scale="0.001 0.001 0.001"/>
     </geometry>
     <material name="silver"/>
@@ -235,5 +235,5 @@
     <origin xyz="-0.047554 -0.0 -0.035941" rpy="0 0 0"/>
     <geometry>
-      <mesh filename="package://clyde_description/src/meshes/servo_neck__1.stl" scale="0.001 0.001 0.001"/>
+      <mesh filename="file://$(find clyde_description)/src/models/clyde_model/meshes/servo_neck__1.stl" scale="0.001 0.001 0.001"/>
     </geometry>
   </collision>
@@ -248,5 +248,5 @@
     <origin xyz="-0.02915 0.052607 -0.02028" rpy="0 0 0"/>
     <geometry>
-      <mesh filename="package://clyde_description/src/meshes/tube__1.stl" scale="0.001 0.001 0.001"/>
+      <mesh filename="file://$(find clyde_description)/src/models/clyde_model/meshes/tube__1.stl" scale="0.001 0.001 0.001"/>
     </geometry>
     <material name="silver"/>
@@ -255,5 +255,5 @@
     <origin xyz="-0.02915 0.052607 -0.02028" rpy="0 0 0"/>
     <geometry>
-      <mesh filename="package://clyde_description/src/meshes/tube__1.stl" scale="0.001 0.001 0.001"/>
+      <mesh filename="file://$(find clyde_description)/src/models/clyde_model/meshes/tube__1.stl" scale="0.001 0.001 0.001"/>
     </geometry>
   </collision>
@@ -268,5 +268,5 @@
     <origin xyz="-0.0525 0.0508 -0.022" rpy="0 0 0"/>
     <geometry>
-      <mesh filename="package://clyde_description/src/meshes/th_rf_1.stl" scale="0.001 0.001 0.001"/>
+      <mesh filename="file://$(find clyde_description)/src/models/clyde_model/meshes/th_rf_1.stl" scale="0.001 0.001 0.001"/>
     </geometry>
     <material name="silver"/>
@@ -275,5 +275,5 @@
     <origin xyz="-0.0525 0.0508 -0.022" rpy="0 0 0"/>
     <geometry>
-      <mesh filename="package://clyde_description/src/meshes/th_rf_1.stl" scale="0.001 0.001 0.001"/>
+      <mesh filename="file://$(find clyde_description)/src/models/clyde_model/meshes/th_rf_1.stl" scale="0.001 0.001 0.001"/>
     </geometry>
   </collision>
@@ -288,5 +288,5 @@
     <origin xyz="-0.008067 0.054937 -0.010094" rpy="0 0 0"/>
     <geometry>
-      <mesh filename="package://clyde_description/src/meshes/c_thorf_1.stl" scale="0.001 0.001 0.001"/>
+      <mesh filename="file://$(find clyde_description)/src/models/clyde_model/meshes/c_thorf_1.stl" scale="0.001 0.001 0.001"/>
     </geometry>
     <material name="silver"/>
@@ -295,5 +295,5 @@
     <origin xyz="-0.008067 0.054937 -0.010094" rpy="0 0 0"/>
     <geometry>
-      <mesh filename="package://clyde_description/src/meshes/c_thorf_1.stl" scale="0.001 0.001 0.001"/>
+      <mesh filename="file://$(find clyde_description)/src/models/clyde_model/meshes/c_thorf_1.stl" scale="0.001 0.001 0.001"/>
     </geometry>
   </collision>
@@ -308,5 +308,5 @@
     <origin xyz="-0.059645 -0.036 -0.017875" rpy="0 0 0"/>
     <geometry>
-      <mesh filename="package://clyde_description/src/meshes/servo_lfs_1.stl" scale="0.001 0.001 0.001"/>
+      <mesh filename="file://$(find clyde_description)/src/models/clyde_model/meshes/servo_lfs_1.stl" scale="0.001 0.001 0.001"/>
     </geometry>
     <material name="silver"/>
@@ -315,5 +315,5 @@
     <origin xyz="-0.059645 -0.036 -0.017875" rpy="0 0 0"/>
     <geometry>
-      <mesh filename="package://clyde_description/src/meshes/servo_lfs_1.stl" scale="0.001 0.001 0.001"/>
+      <mesh filename="file://$(find clyde_description)/src/models/clyde_model/meshes/servo_lfs_1.stl" scale="0.001 0.001 0.001"/>
     </geometry>
   </collision>
@@ -328,5 +328,5 @@
     <origin xyz="0.059645 -0.036 -0.017875" rpy="0 0 0"/>
     <geometry>
-      <mesh filename="package://clyde_description/src/meshes/servo_lrs__1.stl" scale="0.001 0.001 0.001"/>
+      <mesh filename="file://$(find clyde_description)/src/models/clyde_model/meshes/servo_lrs__1.stl" scale="0.001 0.001 0.001"/>
     </geometry>
     <material name="silver"/>
@@ -335,5 +335,5 @@
     <origin xyz="0.059645 -0.036 -0.017875" rpy="0 0 0"/>
     <geometry>
-      <mesh filename="package://clyde_description/src/meshes/servo_lrs__1.stl" scale="0.001 0.001 0.001"/>
+      <mesh filename="file://$(find clyde_description)/src/models/clyde_model/meshes/servo_lrs__1.stl" scale="0.001 0.001 0.001"/>
     </geometry>
   </collision>
@@ -348,5 +348,5 @@
     <origin xyz="-0.0525 0.0485 -0.022" rpy="0 0 0"/>
     <geometry>
-      <mesh filename="package://clyde_description/src/meshes/c_thrf__1.stl" scale="0.001 0.001 0.001"/>
+      <mesh filename="file://$(find clyde_description)/src/models/clyde_model/meshes/c_thrf__1.stl" scale="0.001 0.001 0.001"/>
     </geometry>
     <material name="silver"/>
@@ -355,5 +355,5 @@
     <origin xyz="-0.0525 0.0485 -0.022" rpy="0 0 0"/>
     <geometry>
-      <mesh filename="package://clyde_description/src/meshes/c_thrf__1.stl" scale="0.001 0.001 0.001"/>
+      <mesh filename="file://$(find clyde_description)/src/models/clyde_model/meshes/c_thrf__1.stl" scale="0.001 0.001 0.001"/>
     </geometry>
   </collision>
@@ -368,5 +368,5 @@
     <origin xyz="0.000151 0.03958 -0.010813" rpy="0 0 0"/>
     <geometry>
-      <mesh filename="package://clyde_description/src/meshes/shank_rf_1.stl" scale="0.001 0.001 0.001"/>
+      <mesh filename="file://$(find clyde_description)/src/models/clyde_model/meshes/shank_rf_1.stl" scale="0.001 0.001 0.001"/>
     </geometry>
     <material name="silver"/>
@@ -375,5 +375,5 @@
     <origin xyz="0.000151 0.03958 -0.010813" rpy="0 0 0"/>
     <geometry>
-      <mesh filename="package://clyde_description/src/meshes/shank_rf_1.stl" scale="0.001 0.001 0.001"/>
+      <mesh filename="file://$(find clyde_description)/src/models/clyde_model/meshes/shank_rf_1.stl" scale="0.001 0.001 0.001"/>
     </geometry>
   </collision>
@@ -388,5 +388,5 @@
     <origin xyz="-0.008067 0.04708 -0.010094" rpy="0 0 0"/>
     <geometry>
-      <mesh filename="package://clyde_description/src/meshes/servos_rf_1.stl" scale="0.001 0.001 0.001"/>
+      <mesh filename="file://$(find clyde_description)/src/models/clyde_model/meshes/servos_rf_1.stl" scale="0.001 0.001 0.001"/>
     </geometry>
     <material name="silver"/>
@@ -395,5 +395,5 @@
     <origin xyz="-0.008067 0.04708 -0.010094" rpy="0 0 0"/>
     <geometry>
-      <mesh filename="package://clyde_description/src/meshes/servos_rf_1.stl" scale="0.001 0.001 0.001"/>
+      <mesh filename="file://$(find clyde_description)/src/models/clyde_model/meshes/servos_rf_1.stl" scale="0.001 0.001 0.001"/>
     </geometry>
   </collision>
@@ -408,5 +408,5 @@
     <origin xyz="0.066023 0.050355 -0.018377" rpy="0 0 0"/>
     <geometry>
-      <mesh filename="package://clyde_description/src/meshes/tho_rr_1.stl" scale="0.001 0.001 0.001"/>
+      <mesh filename="file://$(find clyde_description)/src/models/clyde_model/meshes/tho_rr_1.stl" scale="0.001 0.001 0.001"/>
     </geometry>
     <material name="silver"/>
@@ -415,5 +415,5 @@
     <origin xyz="0.066023 0.050355 -0.018377" rpy="0 0 0"/>
     <geometry>
-      <mesh filename="package://clyde_description/src/meshes/tho_rr_1.stl" scale="0.001 0.001 0.001"/>
+      <mesh filename="file://$(find clyde_description)/src/models/clyde_model/meshes/tho_rr_1.stl" scale="0.001 0.001 0.001"/>
     </geometry>
   </collision>
@@ -428,5 +428,5 @@
     <origin xyz="0.07585 0.052607 -0.02028" rpy="0 0 0"/>
     <geometry>
-      <mesh filename="package://clyde_description/src/meshes/tube_rr_1.stl" scale="0.001 0.001 0.001"/>
+      <mesh filename="file://$(find clyde_description)/src/models/clyde_model/meshes/tube_rr_1.stl" scale="0.001 0.001 0.001"/>
     </geometry>
     <material name="silver"/>
@@ -435,5 +435,5 @@
     <origin xyz="0.07585 0.052607 -0.02028" rpy="0 0 0"/>
     <geometry>
-      <mesh filename="package://clyde_description/src/meshes/tube_rr_1.stl" scale="0.001 0.001 0.001"/>
+      <mesh filename="file://$(find clyde_description)/src/models/clyde_model/meshes/tube_rr_1.stl" scale="0.001 0.001 0.001"/>
     </geometry>
   </collision>
@@ -448,5 +448,5 @@
     <origin xyz="0.0525 0.0508 -0.022" rpy="0 0 0"/>
     <geometry>
-      <mesh filename="package://clyde_description/src/meshes/th_rr_1.stl" scale="0.001 0.001 0.001"/>
+      <mesh filename="file://$(find clyde_description)/src/models/clyde_model/meshes/th_rr_1.stl" scale="0.001 0.001 0.001"/>
     </geometry>
     <material name="silver"/>
@@ -455,5 +455,5 @@
     <origin xyz="0.0525 0.0508 -0.022" rpy="0 0 0"/>
     <geometry>
-      <mesh filename="package://clyde_description/src/meshes/th_rr_1.stl" scale="0.001 0.001 0.001"/>
+      <mesh filename="file://$(find clyde_description)/src/models/clyde_model/meshes/th_rr_1.stl" scale="0.001 0.001 0.001"/>
     </geometry>
   </collision>
@@ -468,5 +468,5 @@
     <origin xyz="0.096933 0.054937 -0.010094" rpy="0 0 0"/>
     <geometry>
-      <mesh filename="package://clyde_description/src/meshes/c_thorr_1.stl" scale="0.001 0.001 0.001"/>
+      <mesh filename="file://$(find clyde_description)/src/models/clyde_model/meshes/c_thorr_1.stl" scale="0.001 0.001 0.001"/>
     </geometry>
     <material name="silver"/>
@@ -475,5 +475,5 @@
     <origin xyz="0.096933 0.054937 -0.010094" rpy="0 0 0"/>
     <geometry>
-      <mesh filename="package://clyde_description/src/meshes/c_thorr_1.stl" scale="0.001 0.001 0.001"/>
+      <mesh filename="file://$(find clyde_description)/src/models/clyde_model/meshes/c_thorr_1.stl" scale="0.001 0.001 0.001"/>
     </geometry>
   </collision>
@@ -488,5 +488,5 @@
     <origin xyz="0.105151 0.03958 -0.010813" rpy="0 0 0"/>
     <geometry>
-      <mesh filename="package://clyde_description/src/meshes/shank_rr_1.stl" scale="0.001 0.001 0.001"/>
+      <mesh filename="file://$(find clyde_description)/src/models/clyde_model/meshes/shank_rr_1.stl" scale="0.001 0.001 0.001"/>
     </geometry>
     <material name="silver"/>
@@ -495,5 +495,5 @@
     <origin xyz="0.105151 0.03958 -0.010813" rpy="0 0 0"/>
     <geometry>
-      <mesh filename="package://clyde_description/src/meshes/shank_rr_1.stl" scale="0.001 0.001 0.001"/>
+      <mesh filename="file://$(find clyde_description)/src/models/clyde_model/meshes/shank_rr_1.stl" scale="0.001 0.001 0.001"/>
     </geometry>
   </collision>
@@ -508,5 +508,5 @@
     <origin xyz="0.0525 0.0485 -0.022" rpy="0 0 0"/>
     <geometry>
-      <mesh filename="package://clyde_description/src/meshes/c_thrr_1.stl" scale="0.001 0.001 0.001"/>
+      <mesh filename="file://$(find clyde_description)/src/models/clyde_model/meshes/c_thrr_1.stl" scale="0.001 0.001 0.001"/>
     </geometry>
     <material name="silver"/>
@@ -515,5 +515,5 @@
     <origin xyz="0.0525 0.0485 -0.022" rpy="0 0 0"/>
     <geometry>
-      <mesh filename="package://clyde_description/src/meshes/c_thrr_1.stl" scale="0.001 0.001 0.001"/>
+      <mesh filename="file://$(find clyde_description)/src/models/clyde_model/meshes/c_thrr_1.stl" scale="0.001 0.001 0.001"/>
     </geometry>
   </collision>
@@ -528,5 +528,5 @@
     <origin xyz="0.096933 0.04708 -0.010094" rpy="0 0 0"/>
     <geometry>
-      <mesh filename="package://clyde_description/src/meshes/servos_rr_1.stl" scale="0.001 0.001 0.001"/>
+      <mesh filename="file://$(find clyde_description)/src/models/clyde_model/meshes/servos_rr_1.stl" scale="0.001 0.001 0.001"/>
     </geometry>
     <material name="silver"/>
@@ -535,5 +535,5 @@
     <origin xyz="0.096933 0.04708 -0.010094" rpy="0 0 0"/>
     <geometry>
-      <mesh filename="package://clyde_description/src/meshes/servos_rr_1.stl" scale="0.001 0.001 0.001"/>
+      <mesh filename="file://$(find clyde_description)/src/models/clyde_model/meshes/servos_rr_1.stl" scale="0.001 0.001 0.001"/>
     </geometry>
   </collision>
@@ -548,5 +548,5 @@
     <origin xyz="-0.038977 -0.050355 -0.018377" rpy="0 0 0"/>
     <geometry>
-      <mesh filename="package://clyde_description/src/meshes/tho_lf_1.stl" scale="0.001 0.001 0.001"/>
+      <mesh filename="file://$(find clyde_description)/src/models/clyde_model/meshes/tho_lf_1.stl" scale="0.001 0.001 0.001"/>
     </geometry>
     <material name="silver"/>
@@ -555,5 +555,5 @@
     <origin xyz="-0.038977 -0.050355 -0.018377" rpy="0 0 0"/>
     <geometry>
-      <mesh filename="package://clyde_description/src/meshes/tho_lf_1.stl" scale="0.001 0.001 0.001"/>
+      <mesh filename="file://$(find clyde_description)/src/models/clyde_model/meshes/tho_lf_1.stl" scale="0.001 0.001 0.001"/>
     </geometry>
   </collision>
@@ -568,5 +568,5 @@
     <origin xyz="-0.02915 -0.052607 -0.02028" rpy="0 0 0"/>
     <geometry>
-      <mesh filename="package://clyde_description/src/meshes/tube_lf_1.stl" scale="0.001 0.001 0.001"/>
+      <mesh filename="file://$(find clyde_description)/src/models/clyde_model/meshes/tube_lf_1.stl" scale="0.001 0.001 0.001"/>
     </geometry>
     <material name="silver"/>
@@ -575,5 +575,5 @@
     <origin xyz="-0.02915 -0.052607 -0.02028" rpy="0 0 0"/>
     <geometry>
-      <mesh filename="package://clyde_description/src/meshes/tube_lf_1.stl" scale="0.001 0.001 0.001"/>
+      <mesh filename="file://$(find clyde_description)/src/models/clyde_model/meshes/tube_lf_1.stl" scale="0.001 0.001 0.001"/>
     </geometry>
   </collision>
@@ -588,5 +588,5 @@
     <origin xyz="-0.0525 -0.0508 -0.022" rpy="0 0 0"/>
     <geometry>
-      <mesh filename="package://clyde_description/src/meshes/th_lf_1.stl" scale="0.001 0.001 0.001"/>
+      <mesh filename="file://$(find clyde_description)/src/models/clyde_model/meshes/th_lf_1.stl" scale="0.001 0.001 0.001"/>
     </geometry>
     <material name="silver"/>
@@ -595,5 +595,5 @@
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