Commit message: creating launch to spawn in world

File: src/clyde_description/src/urdf/clyde_simple_without_xacro.urdf (robot description, URDF)
Before this commit: robot clyde, 44 links, 43 joints
Links:
- link base_link: geometry collision mesh filename=package://clyde_description/src/models/clyde_model/meshes/b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 scale=0.001 0.001 0.001; visual mesh filename=package://clyde_description/src/models/clyde_model/meshes/b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 scale=0.001 0.001 0.001
- link battery_1: geometry collision mesh filename=package://clyde_description/src/models/clyde_model/meshes/b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 scale=0.001 0.001 0.001; visual mesh filename=package://clyde_description/src/models/clyde_model/meshes/b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 scale=0.001 0.001 0.001
- link c_neck__1: geometry collision mesh filename=package://clyde_description/src/models/clyde_model/meshes/c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 scale=0.001 0.001 0.001; visual mesh filename=package://clyde_description/src/models/clyde_model/meshes/c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 scale=0.001 0.001 0.001
- link c_thlf_1: geometry collision mesh filename=package://clyde_description/src/models/clyde_model/meshes/c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 scale=0.001 0.001 0.001; visual mesh filename=package://clyde_description/src/models/clyde_model/meshes/c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 scale=0.001 0.001 0.001
- link c_thlr_1: geometry collision mesh filename=package://clyde_description/src/models/clyde_model/meshes/c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 scale=0.001 0.001 0.001; visual mesh filename=package://clyde_description/src/models/clyde_model/meshes/c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 scale=0.001 0.001 0.001
- link c_tholf_1: geometry collision mesh filename=package://clyde_description/src/models/clyde_model/meshes/c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 scale=0.001 0.001 0.001; visual mesh filename=package://clyde_description/src/models/clyde_model/meshes/c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 scale=0.001 0.001 0.001
- link c_tholr__1: geometry collision mesh filename=package://clyde_description/src/models/clyde_model/meshes/c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 scale=0.001 0.001 0.001; visual mesh filename=package://clyde_description/src/models/clyde_model/meshes/c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 scale=0.001 0.001 0.001
- link c_thorf_1: geometry collision mesh filename=package://clyde_description/src/models/clyde_model/meshes/c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 scale=0.001 0.001 0.001; visual mesh filename=package://clyde_description/src/models/clyde_model/meshes/c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 scale=0.001 0.001 0.001
- link c_thorr_1: geometry collision mesh filename=package://clyde_description/src/models/clyde_model/meshes/c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 scale=0.001 0.001 0.001; visual mesh filename=package://clyde_description/src/models/clyde_model/meshes/c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 scale=0.001 0.001 0.001
- link c_thrf__1: geometry collision mesh filename=package://clyde_description/src/models/clyde_model/meshes/c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 scale=0.001 0.001 0.001; visual mesh filename=package://clyde_description/src/models/clyde_model/meshes/c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 scale=0.001 0.001 0.001
- link c_thrr_1: geometry collision mesh filename=package://clyde_description/src/models/clyde_model/meshes/c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 scale=0.001 0.001 0.001; visual mesh filename=package://clyde_description/src/models/clyde_model/meshes/c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 scale=0.001 0.001 0.001
- link cover_1: geometry collision mesh filename=package://clyde_description/src/models/clyde_model/meshes/c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 scale=0.001 0.001 0.001; visual mesh filename=package://clyde_description/src/models/clyde_model/meshes/c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 scale=0.001 0.001 0.001
- link front__1: geometry collision mesh filename=package://clyde_description/src/models/clyde_model/meshes/f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 scale=0.001 0.001 0.001; visual mesh filename=package://clyde_description/src/models/clyde_model/meshes/f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 scale=0.001 0.001 0.001
- link head__1: geometry collision mesh filename=package://clyde_description/src/models/clyde_model/meshes/h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 scale=0.001 0.001 0.001; visual mesh filename=package://clyde_description/src/models/clyde_model/meshes/h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 scale=0.001 0.001 0.001
- link jaw_1: geometry collision mesh filename=package://clyde_description/src/models/clyde_model/meshes/j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 scale=0.001 0.001 0.001; visual mesh filename=package://clyde_description/src/models/clyde_model/meshes/j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 scale=0.001 0.001 0.001
- link rear__1: geometry collision mesh filename=package://clyde_description/src/models/clyde_model/meshes/r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 scale=0.001 0.001 0.001; visual mesh filename=package://clyde_description/src/models/clyde_model/meshes/r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 scale=0.001 0.001 0.001
- link servo_lfs_1: geometry collision mesh filename=package://clyde_description/src/models/clyde_model/meshes/s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 scale=0.001 0.001 0.001; visual mesh filename=package://clyde_description/src/models/clyde_model/meshes/s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 scale=0.001 0.001 0.001
- link servo_lrs__1: geometry collision mesh filename=package://clyde_description/src/models/clyde_model/meshes/s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 scale=0.001 0.001 0.001; visual mesh filename=package://clyde_description/src/models/clyde_model/meshes/s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 scale=0.001 0.001 0.001
- link servo_neck__1: geometry collision mesh filename=package://clyde_description/src/models/clyde_model/meshes/s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 scale=0.001 0.001 0.001; visual mesh filename=package://clyde_description/src/models/clyde_model/meshes/s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 scale=0.001 0.001 0.001
- link servo_rfs_1: geometry collision mesh filename=package://clyde_description/src/models/clyde_model/meshes/s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 scale=0.001 0.001 0.001; visual mesh filename=package://clyde_description/src/models/clyde_model/meshes/s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 scale=0.001 0.001 0.001
- link servo_rrs__1: geometry collision mesh filename=package://clyde_description/src/models/clyde_model/meshes/s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 scale=0.001 0.001 0.001; visual mesh filename=package://clyde_description/src/models/clyde_model/meshes/s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 scale=0.001 0.001 0.001
- link servos_lf_1: geometry collision mesh filename=package://clyde_description/src/models/clyde_model/meshes/s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 scale=0.001 0.001 0.001; visual mesh filename=package://clyde_description/src/models/clyde_model/meshes/s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 scale=0.001 0.001 0.001
- link servos_lr_1: geometry collision mesh filename=package://clyde_description/src/models/clyde_model/meshes/s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 scale=0.001 0.001 0.001; visual mesh filename=package://clyde_description/src/models/clyde_model/meshes/s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 scale=0.001 0.001 0.001
- link servos_rf_1: geometry collision mesh filename=package://clyde_description/src/models/clyde_model/meshes/s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 scale=0.001 0.001 0.001; visual mesh filename=package://clyde_description/src/models/clyde_model/meshes/s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 scale=0.001 0.001 0.001
- link servos_rr_1: geometry collision mesh filename=package://clyde_description/src/models/clyde_model/meshes/s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 scale=0.001 0.001 0.001; visual mesh filename=package://clyde_description/src/models/clyde_model/meshes/s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 scale=0.001 0.001 0.001
- link shank_lf_1: geometry collision mesh filename=package://clyde_description/src/models/clyde_model/meshes/s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 scale=0.001 0.001 0.001; visual mesh filename=package://clyde_description/src/models/clyde_model/meshes/s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 scale=0.001 0.001 0.001
- link shank_lr_1: geometry collision mesh filename=package://clyde_description/src/models/clyde_model/meshes/s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 scale=0.001 0.001 0.001; visual mesh filename=package://clyde_description/src/models/clyde_model/meshes/s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 scale=0.001 0.001 0.001
- link shank_rf_1: geometry collision mesh filename=package://clyde_description/src/models/clyde_model/meshes/s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 scale=0.001 0.001 0.001; visual mesh filename=package://clyde_description/src/models/clyde_model/meshes/s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 scale=0.001 0.001 0.001
- link shank_rr_1: geometry collision mesh filename=package://clyde_description/src/models/clyde_model/meshes/s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 scale=0.001 0.001 0.001; visual mesh filename=package://clyde_description/src/models/clyde_model/meshes/s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 scale=0.001 0.001 0.001
- link th_lf_1: geometry collision mesh filename=package://clyde_description/src/models/clyde_model/meshes/t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 scale=0.001 0.001 0.001; visual mesh filename=package://clyde_description/src/models/clyde_model/meshes/t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 scale=0.001 0.001 0.001
- link th_lr__1: geometry collision mesh filename=package://clyde_description/src/models/clyde_model/meshes/t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 scale=0.001 0.001 0.001; visual mesh filename=package://clyde_description/src/models/clyde_model/meshes/t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 scale=0.001 0.001 0.001
- link th_rf_1: geometry collision mesh filename=package://clyde_description/src/models/clyde_model/meshes/t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 scale=0.001 0.001 0.001; visual mesh filename=package://clyde_description/src/models/clyde_model/meshes/t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 scale=0.001 0.001 0.001
- link th_rr_1: geometry collision mesh filename=package://clyde_description/src/models/clyde_model/meshes/t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 scale=0.001 0.001 0.001; visual mesh filename=package://clyde_description/src/models/clyde_model/meshes/t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 scale=0.001 0.001 0.001
- link tho_lf_1: geometry collision mesh filename=package://clyde_description/src/models/clyde_model/meshes/t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 scale=0.001 0.001 0.001; visual mesh filename=package://clyde_description/src/models/clyde_model/meshes/t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 scale=0.001 0.001 0.001
- link tho_lr_1: geometry collision mesh filename=package://clyde_description/src/models/clyde_model/meshes/t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 scale=0.001 0.001 0.001; visual mesh filename=package://clyde_description/src/models/clyde_model/meshes/t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 scale=0.001 0.001 0.001
- link tho_rf__1: geometry collision mesh filename=package://clyde_description/src/models/clyde_model/meshes/t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 scale=0.001 0.001 0.001; visual mesh filename=package://clyde_description/src/models/clyde_model/meshes/t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 scale=0.001 0.001 0.001
- link tho_rr_1: geometry collision mesh filename=package://clyde_description/src/models/clyde_model/meshes/t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 scale=0.001 0.001 0.001; visual mesh filename=package://clyde_description/src/models/clyde_model/meshes/t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 scale=0.001 0.001 0.001
- link tube__1: geometry collision mesh filename=package://clyde_description/src/models/clyde_model/meshes/t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 scale=0.001 0.001 0.001; visual mesh filename=package://clyde_description/src/models/clyde_model/meshes/t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 scale=0.001 0.001 0.001
- link tube_lf_1: geometry collision mesh filename=package://clyde_description/src/models/clyde_model/meshes/t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 scale=0.001 0.001 0.001; visual mesh filename=package://clyde_description/src/models/clyde_model/meshes/t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 scale=0.001 0.001 0.001
- link tube_lr_1: geometry collision mesh filename=package://clyde_description/src/models/clyde_model/meshes/t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 scale=0.001 0.001 0.001; visual mesh filename=package://clyde_description/src/models/clyde_model/meshes/t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 scale=0.001 0.001 0.001
- link tube_rr_1: geometry collision mesh filename=package://clyde_description/src/models/clyde_model/meshes/t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 scale=0.001 0.001 0.001; visual mesh filename=package://clyde_description/src/models/clyde_model/meshes/t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 scale=0.001 0.001 0.001
