Commit message: changing joint config for straight head

File: src/clyde_description/src/urdf/clyde_simple.urdf (robot description, URDF)
Before this commit: robot clyde, 45 links, 44 joints
Joints:
- joint neck_joint: origin xyz=0.00265 0.0 0.00459 rpy=0 0 0 -> xyz=0.00265 0.0 0.00459 rpy=0.32814212668464987 -0.10093359552132034 0.5922309969483743

File: src/clyde_description/src/urdf/clyde_simple.xacro (robot description, xacro)
@@ -892,5 +892,5 @@
 </joint>
 <joint name="neck_joint" type="continuous">
-  <origin xyz="0.00265 0.0 0.00459" rpy="0 0 0"/>
+  <origin xyz="0.00265 0.0 0.00459" rpy="0.32814212668464987 -0.10093359552132034 0.5922309969483743"/>
   <parent link="c_neck__1"/>
   <child link="servo_neck__1"/>

Commit message: launch file cleanup

File: src/clyde_description/src/urdf/clyde_simple.urdf (robot description, URDF)
Before this commit: robot clyde, 45 links, 44 joints
Links:
- removed link camera_link_optical
- link camera_link: mass None -> 1e-5; geometry collision box size=0.05 0.05 0.05; visual box size=0.05 0.05 0.05
Joints:
- removed joint camera_optical_joint
- joint camera_joint: axis (none) -> 0 1 0; origin xyz=0 0 0 rpy=0 0 0 -> xyz=0.05 0 0 rpy=-0.32814212668464987 0.10093359552132034 -0.5922309969483743
- joint imu_joint: origin xyz=0 0 0.01 -> xyz=0 0 0.03

File: src/clyde_description/src/urdf/clyde_simple.xacro (robot description, xacro)
@@ -4,5 +4,4 @@
 <xacro:include filename="$(find clyde_description)/src/urdf/clyde_simple.trans" />
 <xacro:include filename="$(find clyde_description)/src/urdf/clyde_simple.gazebo" />
-<xacro:include filename="$(find clyde_description)/src/urdf/clyde_cam.xacro" />
 <xacro:macro name="box_inertia" params="m w h d">
   <inertial>
@@ -12,4 +11,5 @@
   </inertial>
 </xacro:macro>
+<xacro:property name="camera_link" value="0.05" />
 <link name="base_link">
   <inertial>
@@ -33,4 +33,30 @@
 </link>
 <link name="base_footprint"/>
+<link name="camera_link">
+  <collision>
+    <origin xyz="0 0 0" rpy="0 0 0"/>
+    <geometry>
+  <box size="${camera_link} ${camera_link} ${camera_link}"/>
+    </geometry>
+  </collision>
+  <visual>
+    <origin xyz="0 0 0" rpy="0 0 0"/>
+    <geometry>
+  <box size="${camera_link} ${camera_link} ${camera_link}"/>
+    </geometry>
+    <material name="red"/>
+  </visual>
+  <inertial>
+    <mass value="1e-5" />
+    <origin xyz="0 0 0" rpy="0 0 0"/>
+    <inertia ixx="1e-6" ixy="0" ixz="0" iyy="1e-6" iyz="0" izz="1e-6" />
+  </inertial>
+</link>
+<joint name="camera_joint" type="fixed">
+  <axis xyz="0 1 0" />
+  <origin xyz="${camera_link} 0 0" rpy="-0.32814212668464987 0.10093359552132034 -0.5922309969483743"/>
+  <parent link="head__1"/>
+  <child link="camera_link"/>
+</joint>
 <link name="front__1">
   <inertial>
@@ -1063,73 +1089,5 @@
   <parent link="base_link"/>
   <child link="imu_link"/>
-  <origin xyz="0 0 0.01"/>
-</joint>
- <gazebo reference="imu_link">
-  <sensor name="imu_sensor" type="imu">
-   <plugin filename="libgazebo_ros_imu_sensor.so" name="imu_plugin">
-      <ros>
-        <namespace>/demo</namespace>
-        <remapping>~/out:=imu</remapping>
-      </ros>
-      <initial_orientation_as_reference>false</initial_orientation_as_reference>
-    </plugin>
-    <always_on>true</always_on>
-    <update_rate>100</update_rate>
-    <visualize>true</visualize>
-    <imu>
-      <angular_velocity>
-        <x>
-          <noise type="gaussian">
-            <mean>0.0</mean>
-            <stddev>2e-4</stddev>
-            <bias_mean>0.0000075</bias_mean>
-            <bias_stddev>0.0000008</bias_stddev>
-          </noise>
-        </x>
-        <y>
-          <noise type="gaussian">
-            <mean>0.0</mean>
-            <stddev>2e-4</stddev>
-            <bias_mean>0.0000075</bias_mean>
-            <bias_stddev>0.0000008</bias_stddev>
-          </noise>
-        </y>
-        <z>
-          <noise type="gaussian">
-            <mean>0.0</mean>
-            <stddev>2e-4</stddev>
-            <bias_mean>0.0000075</bias_mean>
-            <bias_stddev>0.0000008</bias_stddev>
-          </noise>
-        </z>
-      </angular_velocity>
-      <linear_acceleration>
-        <x>
-          <noise type="gaussian">
-            <mean>0.0</mean>
-            <stddev>1.7e-2</stddev>
-            <bias_mean>0.1</bias_mean>
-            <bias_stddev>0.001</bias_stddev>
-          </noise>
-        </x>
-        <y>
-          <noise type="gaussian">
-            <mean>0.0</mean>
-            <stddev>1.7e-2</stddev>
-            <bias_mean>0.1</bias_mean>
-            <bias_stddev>0.001</bias_stddev>
-          </noise>
-        </y>
-        <z>
-          <noise type="gaussian">
-            <mean>0.0</mean>
-            <stddev>1.7e-2</stddev>
-            <bias_mean>0.1</bias_mean>
-            <bias_stddev>0.001</bias_stddev>
-          </noise>
-        </z>
-      </linear_acceleration>
-    </imu>
-  </sensor>
-</gazebo>
+  <origin xyz="0 0 0.03"/>
+</joint>
 </robot>

Commit message: implementing camera visual in gazebo

File: src/clyde_description/src/urdf/clyde_simple.urdf (robot description, URDF)
Before this commit: robot clyde, 44 links, 43 joints
Links:
- added link camera_link_optical
Joints:
- added joint camera_optical_joint: type fixed, parent camera_link, child camera_link_optical, origin xyz=0 0 0 rpy=-1.5707963267948966 0 -1.5707963267948966

File: src/clyde_description/src/urdf/clyde_simple.xacro (robot description, xacro)
@@ -53,4 +53,10 @@
   </inertial>
 </link>
+<joint name="camera_optical_joint" type="fixed">
+    <origin xyz="0 0 0" rpy="${-pi/2} 0 ${-pi/2}" />
+    <parent link="camera_link" />
+    <child link="camera_link_optical" />
+</joint>
+<link name="camera_link_optical"></link>
 <joint name="camera_joint" type="fixed">
   <axis xyz="0 1 0" />
