Commit message: creating testing environments and launch files

File: src/clyde_description/src/urdf/clyde.urdf (robot description, URDF)
Before this commit: robot clyde, 87 links, 86 joints
Links:
- added link dummy
Joints:
- added joint dummy_joint: type fixed, parent dummy, child base_link

File: src/clyde_description/src/urdf/clyde.xacro (robot description, xacro)
@@ -4,7 +4,9 @@
 <xacro:include filename="$(find clyde_description)/src/urdf/clyde.trans" />
 <xacro:include filename="$(find clyde_description)/src/urdf/clyde.gazebo" />
+<link name="dummy">
+</link>
 <link name="base_link">
   <inertial>
-    <origin xyz="0.002168345924058267 4.1430032450566535e-08 0.02555254458454454" rpy="0 0 0"/>
+    <origin xyz="0.002168345924058267 4.1430032450566535e-  08 0.02555254458454454" rpy="0 0 0"/>
     <mass value="0.01989030949409733"/>
     <inertia ixx="1.5e-05" iyy="2.4e-05" izz="3.8e-05" ixy="0.0" iyz="0.0" ixz="-0.0"/>
@@ -24,4 +26,5 @@
   </collision>
 </link>
+<link name="base_footprint"/>
 <link name="front__1">
   <inertial>
@@ -1744,4 +1747,13 @@
   </collision>
 </link>
+<joint name="dummy_joint" type="fixed">
+  <parent link="dummy"/>
+  <child link="base_link"/>
+</joint>
+<joint name="base_joint" type="fixed">
+  <parent link="base_link"/>
+  <child link="base_footprint"/>
+  <origin xyz="0.0 0.0 0.0" rpy="0 0 0"/>
+</joint>
 <joint name="Rigid 1" type="fixed">
   <origin xyz="0.061733 -0.028 0.025792" rpy="0 0 0"/>

Commit message: description implementation with urdf and launch scripts

File: src/clyde_description/src/urdf/clyde.urdf (robot description, URDF)
Before this commit: robot clyde, 88 links, 87 joints
Links:
- added link base_footprint
- added link imu_link, mass 0.1; collision box size=0.1 0.1 0.1; visual box size=0.1 0.1 0.1
Joints:
- added joint base_joint: type fixed, parent base_link, child base_footprint, origin xyz=0.0 0.0 0.0 rpy=0 0 0
- added joint imu_joint: type fixed, parent base_link, child imu_link, origin xyz=0 0 0.01

File: src/clyde_description/src/urdf/clyde.xacro (robot description, xacro)
@@ -4,9 +4,16 @@
 <xacro:include filename="$(find clyde_description)/src/urdf/clyde.trans" />
 <xacro:include filename="$(find clyde_description)/src/urdf/clyde.gazebo" />
+<xacro:macro name="box_inertia" params="m w h d">
+  <inertial>
+    <origin xyz="0 0 0" rpy="${pi/2} 0 ${pi/2}"/>
+    <mass value="${m}"/>
+    <inertia ixx="${(m/12) * (h*h + d*d)}" ixy="0.0" ixz="0.0" iyy="${(m/12) * (w*w + d*d)}" iyz="0.0" izz="${(m/12) * (w*w + h*h)}"/>
+  </inertial>
+</xacro:macro>
 <link name="dummy">
 </link>
 <link name="base_link">
   <inertial>
-    <origin xyz="0.002168345924058267 4.1430032450566535e-  08 0.02555254458454454" rpy="0 0 0"/>
+    <origin xyz="0.002168345924058267 4.1430032450566535e-08 0.02555254458454454" rpy="0 0 0"/>
     <mass value="0.01989030949409733"/>
     <inertia ixx="1.5e-05" iyy="2.4e-05" izz="3.8e-05" ixy="0.0" iyz="0.0" ixz="-0.0"/>
@@ -1746,4 +1753,17 @@
     </geometry>
   </collision>
+</link>
+<link name="imu_link">
+  <visual>
+    <geometry>
+      <box size="0.1 0.1 0.1"/>
+    </geometry>
+  </visual>
+  <collision>
+    <geometry>
+      <box size="0.1 0.1 0.1"/>
+    </geometry>
+  </collision>
+  <xacro:box_inertia m="0.1" w="0.1" d="0.1" h="0.1"/>
 </link>
 <joint name="dummy_joint" type="fixed">
@@ -2195,3 +2215,76 @@
   <child link="screw_8_1"/>
 </joint>
+<joint name="imu_joint" type="fixed">
+  <parent link="base_link"/>
+  <child link="imu_link"/>
+  <origin xyz="0 0 0.01"/>
+</joint>
+ <gazebo reference="imu_link">
+  <sensor name="imu_sensor" type="imu">
+   <plugin filename="libgazebo_ros_imu_sensor.so" name="imu_plugin">
+      <ros>
+        <namespace>/demo</namespace>
+        <remapping>~/out:=imu</remapping>
+      </ros>
+      <initial_orientation_as_reference>false</initial_orientation_as_reference>
+    </plugin>
+    <always_on>true</always_on>
+    <update_rate>100</update_rate>
+    <visualize>true</visualize>
+    <imu>
+      <angular_velocity>
+        <x>
+          <noise type="gaussian">
+            <mean>0.0</mean>
+            <stddev>2e-4</stddev>
+            <bias_mean>0.0000075</bias_mean>
+            <bias_stddev>0.0000008</bias_stddev>
+          </noise>
+        </x>
+        <y>
+          <noise type="gaussian">
+            <mean>0.0</mean>
+            <stddev>2e-4</stddev>
+            <bias_mean>0.0000075</bias_mean>
+            <bias_stddev>0.0000008</bias_stddev>
+          </noise>
+        </y>
+        <z>
+          <noise type="gaussian">
+            <mean>0.0</mean>
+            <stddev>2e-4</stddev>
+            <bias_mean>0.0000075</bias_mean>
+            <bias_stddev>0.0000008</bias_stddev>
+          </noise>
+        </z>
+      </angular_velocity>
+      <linear_acceleration>
+        <x>
+          <noise type="gaussian">
+            <mean>0.0</mean>
+            <stddev>1.7e-2</stddev>
+            <bias_mean>0.1</bias_mean>
+            <bias_stddev>0.001</bias_stddev>
+          </noise>
+        </x>
+        <y>
+          <noise type="gaussian">
+            <mean>0.0</mean>
+            <stddev>1.7e-2</stddev>
+            <bias_mean>0.1</bias_mean>
+            <bias_stddev>0.001</bias_stddev>
+          </noise>
+        </y>
+        <z>
+          <noise type="gaussian">
+            <mean>0.0</mean>
+            <stddev>1.7e-2</stddev>
+            <bias_mean>0.1</bias_mean>
+            <bias_stddev>0.001</bias_stddev>
+          </noise>
+        </z>
+      </linear_acceleration>
+    </imu>
+  </sensor>
+</gazebo>
 </robot>

Commit message: Revert "Nav implementation"

File: src/clyde_description/src/urdf/clyde.urdf (robot description, URDF)
Before this commit: robot clyde, 90 links, 89 joints
Links:
- removed link base_footprint
- removed link imu_link
Joints:
- removed joint base_joint
- removed joint imu_joint

File: src/clyde_description/src/urdf/clyde.xacro (robot description, xacro)
@@ -4,16 +4,9 @@
 <xacro:include filename="$(find clyde_description)/src/urdf/clyde.trans" />
 <xacro:include filename="$(find clyde_description)/src/urdf/clyde.gazebo" />
-<xacro:macro name="box_inertia" params="m w h d">
-  <inertial>
-    <origin xyz="0 0 0" rpy="${pi/2} 0 ${pi/2}"/>
-    <mass value="${m}"/>
-    <inertia ixx="${(m/12) * (h*h + d*d)}" ixy="0.0" ixz="0.0" iyy="${(m/12) * (w*w + d*d)}" iyz="0.0" izz="${(m/12) * (w*w + h*h)}"/>
-  </inertial>
-</xacro:macro>
 <link name="dummy">
 </link>
 <link name="base_link">
   <inertial>
-    <origin xyz="0.002168345924058267 4.1430032450566535e-08 0.02555254458454454" rpy="0 0 0"/>
+    <origin xyz="0.002168345924058267 4.1430032450566535e-  08 0.02555254458454454" rpy="0 0 0"/>
     <mass value="0.01989030949409733"/>
     <inertia ixx="1.5e-05" iyy="2.4e-05" izz="3.8e-05" ixy="0.0" iyz="0.0" ixz="-0.0"/>
@@ -1753,17 +1746,4 @@
     </geometry>
   </collision>
-</link>
-<link name="imu_link">
-  <visual>
-    <geometry>
-      <box size="0.1 0.1 0.1"/>
-    </geometry>
-  </visual>
-  <collision>
-    <geometry>
-      <box size="0.1 0.1 0.1"/>
-    </geometry>
-  </collision>
-  <xacro:box_inertia m="0.1" w="0.1" d="0.1" h="0.1"/>
 </link>
 <joint name="dummy_joint" type="fixed">
@@ -2215,76 +2195,3 @@
   <child link="screw_8_1"/>
 </joint>
-<joint name="imu_joint" type="fixed">
-  <parent link="base_link"/>
-  <child link="imu_link"/>
-  <origin xyz="0 0 0.01"/>
-</joint>
- <gazebo reference="imu_link">
-  <sensor name="imu_sensor" type="imu">
-   <plugin filename="libgazebo_ros_imu_sensor.so" name="imu_plugin">
-      <ros>
-        <namespace>/demo</namespace>
-        <remapping>~/out:=imu</remapping>
-      </ros>
-      <initial_orientation_as_reference>false</initial_orientation_as_reference>
-    </plugin>
-    <always_on>true</always_on>
-    <update_rate>100</update_rate>
-    <visualize>true</visualize>
-    <imu>
-      <angular_velocity>
-        <x>
-          <noise type="gaussian">
-            <mean>0.0</mean>
-            <stddev>2e-4</stddev>
-            <bias_mean>0.0000075</bias_mean>
-            <bias_stddev>0.0000008</bias_stddev>
-          </noise>
-        </x>
-        <y>
-          <noise type="gaussian">
-            <mean>0.0</mean>
-            <stddev>2e-4</stddev>
-            <bias_mean>0.0000075</bias_mean>
-            <bias_stddev>0.0000008</bias_stddev>
-          </noise>
-        </y>
-        <z>
-          <noise type="gaussian">
-            <mean>0.0</mean>
-            <stddev>2e-4</stddev>
-            <bias_mean>0.0000075</bias_mean>
-            <bias_stddev>0.0000008</bias_stddev>
-          </noise>
-        </z>
-      </angular_velocity>
-      <linear_acceleration>
-        <x>
-          <noise type="gaussian">
-            <mean>0.0</mean>
-            <stddev>1.7e-2</stddev>
-            <bias_mean>0.1</bias_mean>
-            <bias_stddev>0.001</bias_stddev>
-          </noise>
-        </x>
-        <y>
-          <noise type="gaussian">
-            <mean>0.0</mean>
-            <stddev>1.7e-2</stddev>
-            <bias_mean>0.1</bias_mean>
-            <bias_stddev>0.001</bias_stddev>
-          </noise>
-        </y>
-        <z>
-          <noise type="gaussian">
-            <mean>0.0</mean>
-            <stddev>1.7e-2</stddev>
-            <bias_mean>0.1</bias_mean>
-            <bias_stddev>0.001</bias_stddev>
-          </noise>
-        </z>
-      </linear_acceleration>
-    </imu>
-  </sensor>
-</gazebo>
 </robot>

File: src/clyde_description/src/urdf/materials.xacro (robot description, xacro)
@@ -4,6 +4,3 @@
   <color rgba="0.700 0.700 0.700 1.000"/>
 </material>
-<material name="red">
-  <color rgba="1.000 0.000 0.000 1.000"/>
-</material>
 </robot>

Commit message: cleaning up urdf and launching in gazebo with sdf

File: src/clyde_description/src/urdf/clyde.urdf (robot description, URDF)
Before this commit: robot clyde, 90 links, 89 joints
Links:
- removed link a_1
- removed link b__1
- removed link c_1
- removed link d_1
- removed link dummy
- removed link e_1
- removed link f_1
- removed link g_1
- removed link h__1
- removed link i_1
- removed link j__1
- removed link k_1
- removed link l_1
- removed link logo_1_1
- removed link logo_2_1
- removed link logo_3_1
- removed link logo_4_1
- removed link logo_5_1
- removed link screw_10_1
- removed link screw_11_1
- removed link screw_12_1
- removed link screw_13_1
- removed link screw_14_1
- removed link screw_15_1
- removed link screw_16_1
- removed link screw_17_1
- removed link screw_18_1
- removed link screw_19_1
- removed link screw_1_1
- removed link screw_20_1
- removed link screw_21_1
- removed link screw_2_1
- removed link screw_3_1
- removed link screw_4_1
- removed link screw_5_1
- removed link screw_6_1
- removed link screw_7_1
- removed link screw_8_1
- removed link screw_9_1
- removed link screwm_1_1
- removed link screwm_2_1
- removed link screwm_3_1
- removed link screwm_4_1
- removed link screwm_5_1
- removed link screwm_6_1
- removed link screwm_7_1
- removed link screwm_8_1
- added link camera_link, mass 1e-5; collision box size=0.01 0.01 0.01; visual box size=0.01 0.01 0.01
- added link camera_link_optical
- link base_link: geometry collision mesh filename=file:///workspaces/clyderos2/install/share/clyde_descriptio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 scale=0.001 0.001 0.001; visual mesh filename=file:///workspaces/clyderos2/install/share/clyde_descriptio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 scale=0.001 0.001 0.001
- link battery_1: geometry collision mesh filename=file:///workspaces/clyderos2/install/share/clyde_descriptio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 scale=0.001 0.001 0.001; visual mesh filename=file:///workspaces/clyderos2/install/share/clyde_descriptio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 scale=0.001 0.001 0.001
- link c_neck__1: geometry collision mesh filename=file:///workspaces/clyderos2/install/share/clyde_descriptio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 scale=0.001 0.001 0.001; visual mesh filename=file:///workspaces/clyderos2/install/share/clyde_descriptio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 scale=0.001 0.001 0.001
- link c_thlf_1: geometry collision mesh filename=file:///workspaces/clyderos2/install/share/clyde_descriptio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 scale=0.001 0.001 0.001; visual mesh filename=file:///workspaces/clyderos2/install/share/clyde_descriptio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 scale=0.001 0.001 0.001
- link c_thlr_1: geometry collision mesh filename=file:///workspaces/clyderos2/install/share/clyde_descriptio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 scale=0.001 0.001 0.001; visual mesh filename=file:///workspaces/clyderos2/install/share/clyde_descriptio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 scale=0.001 0.001 0.001
- link c_tholf_1: geometry collision mesh filename=file:///workspaces/clyderos2/install/share/clyde_descriptio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 scale=0.001 0.001 0.001; visual mesh filename=file:///workspaces/clyderos2/install/share/clyde_descriptio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 scale=0.001 0.001 0.001
- link c_tholr__1: geometry collision mesh filename=file:///workspaces/clyderos2/install/share/clyde_descriptio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 scale=0.001 0.001 0.001; visual mesh filename=file:///workspaces/clyderos2/install/share/clyde_descriptio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 scale=0.001 0.001 0.001
- link c_thorf_1: geometry collision mesh filename=file:///workspaces/clyderos2/install/share/clyde_descriptio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 scale=0.001 0.001 0.001; visual mesh filename=file:///workspaces/clyderos2/install/share/clyde_descriptio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 scale=0.001 0.001 0.001
- link c_thorr_1: geometry collision mesh filename=file:///workspaces/clyderos2/install/share/clyde_descriptio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 scale=0.001 0.001 0.001; visual mesh filename=file:///workspaces/clyderos2/install/share/clyde_descriptio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 scale=0.001 0.001 0.001
- link c_thrf__1: geometry collision mesh filename=file:///workspaces/clyderos2/install/share/clyde_descriptio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 scale=0.001 0.001 0.001; visual mesh filename=file:///workspaces/clyderos2/install/share/clyde_descriptio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 scale=0.001 0.001 0.001
- link c_thrr_1: geometry collision mesh filename=file:///workspaces/clyderos2/install/share/clyde_descriptio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 scale=0.001 0.001 0.001; visual mesh filename=file:///workspaces/clyderos2/install/share/clyde_descriptio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 scale=0.001 0.001 0.001
- link cover_1: geometry collision mesh filename=file:///workspaces/clyderos2/install/share/clyde_descriptio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 scale=0.001 0.001 0.001; visual mesh filename=file:///workspaces/clyderos2/install/share/clyde_descriptio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 scale=0.001 0.001 0.001
- link front__1: geometry collision mesh filename=file:///workspaces/clyderos2/install/share/clyde_descriptio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 scale=0.001 0.001 0.001; visual mesh filename=file:///workspaces/clyderos2/install/share/clyde_descriptio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 scale=0.001 0.001 0.001
- link head__1: geometry collision mesh filename=file:///workspaces/clyderos2/install/share/clyde_descriptio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 scale=0.001 0.001 0.001; visual mesh filename=file:///workspaces/clyderos2/install/share/clyde_descriptio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 scale=0.001 0.001 0.001
- link imu_link: geometry collision box size=0.01 0.01 0.01; visual box size=0.01 0.01 0.01
- link jaw_1: geometry collision mesh filename=file:///workspaces/clyderos2/install/share/clyde_descriptio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 scale=0.001 0.001 0.001; visual mesh filename=file:///workspaces/clyderos2/install/share/clyde_descriptio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 scale=0.001 0.001 0.001
- link rear__1: geometry collision mesh filename=file:///workspaces/clyderos2/install/share/clyde_descriptio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 scale=0.001 0.001 0.001; visual mesh filename=file:///workspaces/clyderos2/install/share/clyde_descriptio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 scale=0.001 0.001 0.001
- link servo_lfs_1: geometry collision mesh filename=file:///workspaces/clyderos2/install/share/clyde_descriptio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 scale=0.001 0.001 0.001; visual mesh filename=file:///workspaces/clyderos2/install/share/clyde_descriptio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 scale=0.001 0.001 0.001
- link servo_lrs__1: geometry collision mesh filename=file:///workspaces/clyderos2/install/share/clyde_descriptio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 scale=0.001 0.001 0.001; visual mesh filename=file:///workspaces/clyderos2/install/share/clyde_descriptio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 scale=0.001 0.001 0.001
- link servo_neck__1: geometry collision mesh filename=file:///workspaces/clyderos2/install/share/clyde_descriptio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 scale=0.001 0.001 0.001; visual mesh filename=file:///workspaces/clyderos2/install/share/clyde_descriptio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 scale=0.001 0.001 0.001
- link servo_rfs_1: geometry collision mesh filename=file:///workspaces/clyderos2/install/share/clyde_descriptio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 scale=0.001 0.001 0.001; visual mesh filename=file:///workspaces/clyderos2/install/share/clyde_descriptio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 scale=0.001 0.001 0.001
- link servo_rrs__1: geometry collision mesh filename=file:///workspaces/clyderos2/install/share/clyde_descriptio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 scale=0.001 0.001 0.001; visual mesh filename=file:///workspaces/clyderos2/install/share/clyde_descriptio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 scale=0.001 0.001 0.001
- link servos_lf_1: geometry collision mesh filename=file:///workspaces/clyderos2/install/share/clyde_descriptio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 scale=0.001 0.001 0.001; visual mesh filename=file:///workspaces/clyderos2/install/share/clyde_descriptio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 scale=0.001 0.001 0.001
- link servos_lr_1: geometry collision mesh filename=file:///workspaces/clyderos2/install/share/clyde_descriptio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 scale=0.001 0.001 0.001; visual mesh filename=file:///workspaces/clyderos2/install/share/clyde_descriptio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 scale=0.001 0.001 0.001
- link servos_rf_1: geometry collision mesh filename=file:///workspaces/clyderos2/install/share/clyde_descriptio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 scale=0.001 0.001 0.001; visual mesh filename=file:///workspaces/clyderos2/install/share/clyde_descriptio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 scale=0.001 0.001 0.001
- link servos_rr_1: geometry collision mesh filename=file:///workspaces/clyderos2/install/share/clyde_descriptio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 scale=0.001 0.001 0.001; visual mesh filename=file:///workspaces/clyderos2/install/share/clyde_descriptio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 scale=0.001 0.001 0.001
- link shank_lf_1: geometry collision mesh filename=file:///workspaces/clyderos2/install/share/clyde_descriptio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 scale=0.001 0.001 0.001; visual mesh filename=file:///workspaces/clyderos2/install/share/clyde_descriptio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 scale=0.001 0.001 0.001
- link shank_lr_1: geometry collision mesh filename=file:///workspaces/clyderos2/install/share/clyde_descriptio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 scale=0.001 0.001 0.001; visual mesh filename=file:///workspaces/clyderos2/install/share/clyde_descriptio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 scale=0.001 0.001 0.001
- link shank_rf_1: geometry collision mesh filename=file:///workspaces/clyderos2/install/share/clyde_descriptio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 scale=0.001 0.001 0.001; visual mesh filename=file:///workspaces/clyderos2/install/share/clyde_descriptio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 scale=0.001 0.001 0.001
- link shank_rr_1: geometry collision mesh filename=file:///workspaces/clyderos2/install/share/clyde_descriptio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 scale=0.001 0.001 0.001; visual mesh filename=file:///workspaces/clyderos2/install/share/clyde_descriptio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 scale=0.001 0.001 0.001
- link th_lf_1: geometry collision mesh filename=file:///workspaces/clyderos2/install/share/clyde_descriptio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 scale=0.001 0.001 0.001; visual mesh filename=file:///workspaces/clyderos2/install/share/clyde_descriptio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 scale=0.001 0.001 0.001
- link th_lr__1: geometry collision mesh filename=file:///workspaces/clyderos2/install/share/clyde_descriptio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 scale=0.001 0.001 0.001; visual mesh filename=file:///workspaces/clyderos2/install/share/clyde_descriptio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 scale=0.001 0.001 0.001
- link th_rf_1: geometry collision mesh filename=file:///workspaces/clyderos2/install/share/clyde_descriptio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 scale=0.001 0.001 0.001; visual mesh filename=file:///workspaces/clyderos2/install/share/clyde_descriptio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 scale=0.001 0.001 0.001
- link th_rr_1: geometry collision mesh filename=file:///workspaces/clyderos2/install/share/clyde_descriptio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 scale=0.001 0.001 0.001; visual mesh filename=file:///workspaces/clyderos2/install/share/clyde_descriptio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 scale=0.001 0.001 0.001
- link tho_lf_1: geometry collision mesh filename=file:///workspaces/clyderos2/install/share/clyde_descriptio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 scale=0.001 0.001 0.001; visual mesh filename=file:///workspaces/clyderos2/install/share/clyde_descriptio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 scale=0.001 0.001 0.001
- link tho_lr_1: geometry collision mesh filename=file:///workspaces/clyderos2/install/share/clyde_descriptio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 scale=0.001 0.001 0.001; visual mesh filename=file:///workspaces/clyderos2/install/share/clyde_descriptio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 scale=0.001 0.001 0.001
- link tho_rf__1: geometry collision mesh filename=file:///workspaces/clyderos2/install/share/clyde_descriptio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 scale=0.001 0.001 0.001; visual mesh filename=file:///workspaces/clyderos2/install/share/clyde_descriptio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 scale=0.001 0.001 0.001
- link tho_rr_1: geometry collision mesh filename=file:///workspaces/clyderos2/install/share/clyde_descriptio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 scale=0.001 0.001 0.001; visual mesh filename=file:///workspaces/clyderos2/install/share/clyde_descriptio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 scale=0.001 0.001 0.001
- link tube__1: geometry collision mesh filename=file:///workspaces/clyderos2/install/share/clyde_descriptio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 scale=0.001 0.001 0.001; visual mesh filename=file:///workspaces/clyderos2/install/share/clyde_descriptio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 scale=0.001 0.001 0.001
- link tube_lf_1: geometry collision mesh filename=file:///workspaces/clyderos2/install/share/clyde_descriptio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 scale=0.001 0.001 0.001; visual mesh filename=file:///workspaces/clyderos2/install/share/clyde_descriptio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 scale=0.001 0.001 0.001
- link tube_lr_1: geometry collision mesh filename=file:///workspaces/clyderos2/install/share/clyde_descriptio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 scale=0.001 0.001 0.001; visual mesh filename=file:///workspaces/clyderos2/install/share/clyde_descriptio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 scale=0.001 0.001 0.001
- link tube_rr_1: geometry collision mesh filename=file:///workspaces/clyderos2/install/share/clyde_descriptio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 scale=0.001 0.001 0.001; visual mesh filename=file:///workspaces/clyderos2/install/share/clyde_descriptio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 scale=0.001 0.001 0.001
Joints:
- removed joint Rigid 17
- removed joint Rigid 18
- removed joint Rigid 19
- removed joint Rigid 20
- removed joint Rigid 21
- removed joint Rigid 22
- removed joint Rigid 24
- removed joint Rigid 25
- removed joint Rigid 26
- removed joint Rigid 27
- removed joint Rigid 28
- removed joint Rigid 29
- removed joint Rigid 53
- removed joint Rigid 54
- removed joint Rigid 55
- removed joint Rigid 56
- removed joint Rigid 57
- removed joint Rigid 60
- removed joint Rigid 61
- removed joint Rigid 62
- removed joint Rigid 63
- removed joint Rigid 64
- removed joint Rigid 65
- removed joint Rigid 66
- removed joint Rigid 67
- removed joint Rigid 68
- removed joint Rigid 69
- removed joint Rigid 70
- removed joint Rigid 71
- removed joint Rigid 72
- removed joint Rigid 73
- removed joint Rigid 74
- removed joint Rigid 75
- removed joint Rigid 76
- removed joint Rigid 77
- removed joint Rigid 78
- removed joint Rigid 79
- removed joint Rigid 80
- removed joint Rigid 81
- removed joint Rigid 82
- removed joint Rigid 83
- removed joint Rigid 84
- removed joint Rigid 85
- removed joint Rigid 86
- removed joint Rigid 87
- removed joint Rigid 88
- removed joint dummy_joint
- added joint camera_joint: type fixed, parent head__1, child camera_link, origin xyz=0.01 0.020 0.015 rpy=-0.32814212668464987 0.10093359552132034 -0.5922309969483743, axis 0 1 0
- added joint camera_optical_joint: type fixed, parent camera_link, child camera_link_optical, origin xyz=0 0 0 rpy=-1.5707963267948966 0 -1.5707963267948966
- joint base_joint: child base_footprint -> base_link; parent base_link -> base_footprint
- joint imu_joint: origin xyz=0 0 0.01 -> xyz=0 0 0.03
- joint neck_joint: origin xyz=0.00265 0.0 0.00459 rpy=0 0 0 -> xyz=0.00265 0.0 0.00459 rpy=0.32814212668464987 -0.10093359552132034 0.5922309969483743
