Commit message: cleaning up urdf and launching in gazebo with sdf

File: src/clyde_description/src/urdf/clyde.xacro (robot description, xacro)
@@ -2,6 +2,6 @@
 <robot name="clyde" xmlns:xacro="http://www.ros.org/wiki/xacro">
 <xacro:include filename="$(find clyde_description)/src/urdf/materials.xacro" />
-<xacro:include filename="$(find clyde_description)/src/urdf/clyde.trans" />
-<xacro:include filename="$(find clyde_description)/src/urdf/clyde.gazebo" />
+<xacro:include filename="$(find clyde_description)/src/urdf/clyde_simple.trans" />
+<xacro:include filename="$(find clyde_description)/src/urdf/clyde_simple.gazebo" />
 <xacro:macro name="box_inertia" params="m w h d">
   <inertial>
@@ -11,9 +11,8 @@
   </inertial>
 </xacro:macro>
-<link name="dummy">
-</link>
+<xacro:property name="camera_link" value="0.01" />
 <link name="base_link">
   <inertial>
-    <origin xyz="0.002168345924058267 4.1430032450566535e-08 0.02555254458454454" rpy="0 0 0"/>
+    <origin xyz="0.002168345924058267 0 0.02555254458454454" rpy="0 0 0"/>
     <mass value="0.01989030949409733"/>
     <inertia ixx="1.5e-05" iyy="2.4e-05" izz="3.8e-05" ixy="0.0" iyz="0.0" ixz="-0.0"/>
@@ -22,5 +21,5 @@
     <origin xyz="0 0 0" rpy="0 0 0"/>
     <geometry>
-      <mesh filename="package://clyde_description/src/meshes/base_link.stl" scale="0.001 0.001 0.001"/>
+      <mesh filename="file://$(find clyde_description)/src/models/clyde_model/meshes/base_link.stl" scale="0.001 0.001 0.001"/>
     </geometry>
     <material name="silver"/>
@@ -29,9 +28,41 @@
     <origin xyz="0 0 0" rpy="0 0 0"/>
     <geometry>
-      <mesh filename="package://clyde_description/src/meshes/base_link.stl" scale="0.001 0.001 0.001"/>
+      <mesh filename="file://$(find clyde_description)/src/models/clyde_model/meshes/base_link.stl" scale="0.001 0.001 0.001"/>
     </geometry>
   </collision>
 </link>
 <link name="base_footprint"/>
+<link name="camera_link">
+  <collision>
+    <origin xyz="0 0 0" rpy="0 0 0"/>
+    <geometry>
+  <box size="${camera_link} ${camera_link} ${camera_link}"/>
+    </geometry>
+  </collision>
+  <visual>
+    <origin xyz="0 0 0" rpy="0 0 0"/>
+    <geometry>
+  <box size="${camera_link} ${camera_link} ${camera_link}"/>
+    </geometry>
+    <material name="red"/>
+  </visual>
+  <inertial>
+    <mass value="1e-5" />
+    <origin xyz="0 0 0" rpy="0 0 0"/>
+    <inertia ixx="1e-6" ixy="0" ixz="0" iyy="1e-6" iyz="0" izz="1e-6" />
+  </inertial>
+</link>
+<joint name="camera_optical_joint" type="fixed">
+    <origin xyz="0 0 0" rpy="${-pi/2} 0 ${-pi/2}" />
+    <parent link="camera_link" />
+    <child link="camera_link_optical" />
+</joint>
+<link name="camera_link_optical"></link>
+<joint name="camera_joint" type="fixed">
+  <axis xyz="0 1 0" />
+  <origin xyz="${camera_link} 0.020 0.015" rpy="-0.32814212668464987 0.10093359552132034 -0.5922309969483743"/>
+  <parent link="head__1"/>
+  <child link="camera_link"/>
+</joint>
 <link name="front__1">
   <inertial>
@@ -43,5 +74,5 @@
     <origin xyz="-0.061733 0.028 -0.025792" rpy="0 0 0"/>
     <geometry>
-      <mesh filename="package://clyde_description/src/meshes/front__1.stl" scale="0.001 0.001 0.001"/>
+      <mesh filename="file://$(find clyde_description)/src/models/clyde_model/meshes/front__1.stl" scale="0.001 0.001 0.001"/>
     </geometry>
     <material name="silver"/>
@@ -50,5 +81,5 @@
     <origin xyz="-0.061733 0.028 -0.025792" rpy="0 0 0"/>
     <geometry>
-      <mesh filename="package://clyde_description/src/meshes/front__1.stl" scale="0.001 0.001 0.001"/>
+      <mesh filename="file://$(find clyde_description)/src/models/clyde_model/meshes/front__1.stl" scale="0.001 0.001 0.001"/>
     </geometry>
   </collision>
@@ -63,5 +94,5 @@
     <origin xyz="0.061733 -0.028 -0.025792" rpy="0 0 0"/>
     <geometry>
-      <mesh filename="package://clyde_description/src/meshes/rear__1.stl" scale="0.001 0.001 0.001"/>
+      <mesh filename="file://$(find clyde_description)/src/models/clyde_model/meshes/rear__1.stl" scale="0.001 0.001 0.001"/>
     </geometry>
     <material name="silver"/>
@@ -70,5 +101,5 @@
     <origin xyz="0.061733 -0.028 -0.025792" rpy="0 0 0"/>
     <geometry>
-      <mesh filename="package://clyde_description/src/meshes/rear__1.stl" scale="0.001 0.001 0.001"/>
+      <mesh filename="file://$(find clyde_description)/src/models/clyde_model/meshes/rear__1.stl" scale="0.001 0.001 0.001"/>
     </geometry>
   </collision>
@@ -83,5 +114,5 @@
     <origin xyz="-0.059645 0.036 -0.017875" rpy="0 0 0"/>
     <geometry>
-      <mesh filename="package://clyde_description/src/meshes/servo_rfs_1.stl" scale="0.001 0.001 0.001"/>
+      <mesh filename="file://$(find clyde_description)/src/models/clyde_model/meshes/servo_rfs_1.stl" scale="0.001 0.001 0.001"/>
     </geometry>
     <material name="silver"/>
@@ -90,5 +121,5 @@
     <origin xyz="-0.059645 0.036 -0.017875" rpy="0 0 0"/>
     <geometry>
-      <mesh filename="package://clyde_description/src/meshes/servo_rfs_1.stl" scale="0.001 0.001 0.001"/>
+      <mesh filename="file://$(find clyde_description)/src/models/clyde_model/meshes/servo_rfs_1.stl" scale="0.001 0.001 0.001"/>
     </geometry>
   </collision>
@@ -103,5 +134,5 @@
     <origin xyz="0.059645 0.036 -0.017875" rpy="0 0 0"/>
     <geometry>
-      <mesh filename="package://clyde_description/src/meshes/servo_rrs__1.stl" scale="0.001 0.001 0.001"/>
+      <mesh filename="file://$(find clyde_description)/src/models/clyde_model/meshes/servo_rrs__1.stl" scale="0.001 0.001 0.001"/>
     </geometry>
     <material name="silver"/>
@@ -110,5 +141,5 @@
     <origin xyz="0.059645 0.036 -0.017875" rpy="0 0 0"/>
     <geometry>
-      <mesh filename="package://clyde_description/src/meshes/servo_rrs__1.stl" scale="0.001 0.001 0.001"/>
+      <mesh filename="file://$(find clyde_description)/src/models/clyde_model/meshes/servo_rrs__1.stl" scale="0.001 0.001 0.001"/>
     </geometry>
   </collision>
@@ -123,5 +154,5 @@
     <origin xyz="-0.044904 -0.0 -0.031351" rpy="0 0 0"/>
     <geometry>
-      <mesh filename="package://clyde_description/src/meshes/c_neck__1.stl" scale="0.001 0.001 0.001"/>
+      <mesh filename="file://$(find clyde_description)/src/models/clyde_model/meshes/c_neck__1.stl" scale="0.001 0.001 0.001"/>
     </geometry>
     <material name="silver"/>
@@ -130,5 +161,5 @@
     <origin xyz="-0.044904 -0.0 -0.031351" rpy="0 0 0"/>
     <geometry>
-      <mesh filename="package://clyde_description/src/meshes/c_neck__1.stl" scale="0.001 0.001 0.001"/>
+      <mesh filename="file://$(find clyde_description)/src/models/clyde_model/meshes/c_neck__1.stl" scale="0.001 0.001 0.001"/>
     </geometry>
   </collision>
@@ -143,5 +174,5 @@
     <origin xyz="-0.055711 0.017155 -0.060327" rpy="0 0 0"/>
     <geometry>
-      <mesh filename="package://clyde_description/src/meshes/head__1.stl" scale="0.001 0.001 0.001"/>
+      <mesh filename="file://$(find clyde_description)/src/models/clyde_model/meshes/head__1.stl" scale="0.001 0.001 0.001"/>
     </geometry>
     <material name="silver"/>
@@ -150,5 +181,5 @@
     <origin xyz="-0.055711 0.017155 -0.060327" rpy="0 0 0"/>
     <geometry>
-      <mesh filename="package://clyde_description/src/meshes/head__1.stl" scale="0.001 0.001 0.001"/>
+      <mesh filename="file://$(find clyde_description)/src/models/clyde_model/meshes/head__1.stl" scale="0.001 0.001 0.001"/>
     </geometry>
   </collision>
@@ -163,5 +194,5 @@
     <origin xyz="-0.06445 0.012925 -0.034027" rpy="0 0 0"/>
     <geometry>
-      <mesh filename="package://clyde_description/src/meshes/jaw_1.stl" scale="0.001 0.001 0.001"/>
+      <mesh filename="file://$(find clyde_description)/src/models/clyde_model/meshes/jaw_1.stl" scale="0.001 0.001 0.001"/>
     </geometry>
     <material name="silver"/>
@@ -170,5 +201,5 @@
     <origin xyz="-0.06445 0.012925 -0.034027" rpy="0 0 0"/>
     <geometry>
-      <mesh filename="package://clyde_description/src/meshes/jaw_1.stl" scale="0.001 0.001 0.001"/>
+      <mesh filename="file://$(find clyde_description)/src/models/clyde_model/meshes/jaw_1.stl" scale="0.001 0.001 0.001"/>
     </geometry>
   </collision>
@@ -183,5 +214,5 @@
     <origin xyz="-0.038977 0.050355 -0.018377" rpy="0 0 0"/>
     <geometry>
-      <mesh filename="package://clyde_description/src/meshes/tho_rf__1.stl" scale="0.001 0.001 0.001"/>
+      <mesh filename="file://$(find clyde_description)/src/models/clyde_model/meshes/tho_rf__1.stl" scale="0.001 0.001 0.001"/>
     </geometry>
     <material name="silver"/>
@@ -190,5 +221,5 @@
     <origin xyz="-0.038977 0.050355 -0.018377" rpy="0 0 0"/>
     <geometry>
-      <mesh filename="package://clyde_description/src/meshes/tho_rf__1.stl" scale="0.001 0.001 0.001"/>
+      <mesh filename="file://$(find clyde_description)/src/models/clyde_model/meshes/tho_rf__1.stl" scale="0.001 0.001 0.001"/>
     </geometry>
   </collision>
@@ -203,5 +234,5 @@
     <origin xyz="-0.047554 -0.0 -0.035941" rpy="0 0 0"/>
     <geometry>
-      <mesh filename="package://clyde_description/src/meshes/servo_neck__1.stl" scale="0.001 0.001 0.001"/>
+      <mesh filename="file://$(find clyde_description)/src/models/clyde_model/meshes/servo_neck__1.stl" scale="0.001 0.001 0.001"/>
     </geometry>
     <material name="silver"/>
@@ -210,5 +241,5 @@
     <origin xyz="-0.047554 -0.0 -0.035941" rpy="0 0 0"/>
     <geometry>
-      <mesh filename="package://clyde_description/src/meshes/servo_neck__1.stl" scale="0.001 0.001 0.001"/>
+      <mesh filename="file://$(find clyde_description)/src/models/clyde_model/meshes/servo_neck__1.stl" scale="0.001 0.001 0.001"/>
     </geometry>
   </collision>
@@ -223,5 +254,5 @@
     <origin xyz="-0.02915 0.052607 -0.02028" rpy="0 0 0"/>
     <geometry>
-      <mesh filename="package://clyde_description/src/meshes/tube__1.stl" scale="0.001 0.001 0.001"/>
+      <mesh filename="file://$(find clyde_description)/src/models/clyde_model/meshes/tube__1.stl" scale="0.001 0.001 0.001"/>
     </geometry>
     <material name="silver"/>
@@ -230,5 +261,5 @@
     <origin xyz="-0.02915 0.052607 -0.02028" rpy="0 0 0"/>
     <geometry>
-      <mesh filename="package://clyde_description/src/meshes/tube__1.stl" scale="0.001 0.001 0.001"/>
+      <mesh filename="file://$(find clyde_description)/src/models/clyde_model/meshes/tube__1.stl" scale="0.001 0.001 0.001"/>
     </geometry>
   </collision>
@@ -243,5 +274,5 @@
     <origin xyz="-0.0525 0.0508 -0.022" rpy="0 0 0"/>
     <geometry>
-      <mesh filename="package://clyde_description/src/meshes/th_rf_1.stl" scale="0.001 0.001 0.001"/>
+      <mesh filename="file://$(find clyde_description)/src/models/clyde_model/meshes/th_rf_1.stl" scale="0.001 0.001 0.001"/>
     </geometry>
     <material name="silver"/>
@@ -250,5 +281,5 @@
     <origin xyz="-0.0525 0.0508 -0.022" rpy="0 0 0"/>
     <geometry>
-      <mesh filename="package://clyde_description/src/meshes/th_rf_1.stl" scale="0.001 0.001 0.001"/>
+      <mesh filename="file://$(find clyde_description)/src/models/clyde_model/meshes/th_rf_1.stl" scale="0.001 0.001 0.001"/>
     </geometry>
   </collision>
@@ -263,5 +294,5 @@
     <origin xyz="-0.008067 0.054937 -0.010094" rpy="0 0 0"/>
     <geometry>
-      <mesh filename="package://clyde_description/src/meshes/c_thorf_1.stl" scale="0.001 0.001 0.001"/>
+      <mesh filename="file://$(find clyde_description)/src/models/clyde_model/meshes/c_thorf_1.stl" scale="0.001 0.001 0.001"/>
     </geometry>
     <material name="silver"/>
@@ -270,5 +301,5 @@
     <origin xyz="-0.008067 0.054937 -0.010094" rpy="0 0 0"/>
     <geometry>
-      <mesh filename="package://clyde_description/src/meshes/c_thorf_1.stl" scale="0.001 0.001 0.001"/>
+      <mesh filename="file://$(find clyde_description)/src/models/clyde_model/meshes/c_thorf_1.stl" scale="0.001 0.001 0.001"/>
     </geometry>
   </collision>
@@ -283,5 +314,5 @@
     <origin xyz="-0.059645 -0.036 -0.017875" rpy="0 0 0"/>
     <geometry>
-      <mesh filename="package://clyde_description/src/meshes/servo_lfs_1.stl" scale="0.001 0.001 0.001"/>
+      <mesh filename="file://$(find clyde_description)/src/models/clyde_model/meshes/servo_lfs_1.stl" scale="0.001 0.001 0.001"/>
     </geometry>
     <material name="silver"/>
@@ -290,5 +321,5 @@
     <origin xyz="-0.059645 -0.036 -0.017875" rpy="0 0 0"/>
     <geometry>
-      <mesh filename="package://clyde_description/src/meshes/servo_lfs_1.stl" scale="0.001 0.001 0.001"/>
+      <mesh filename="file://$(find clyde_description)/src/models/clyde_model/meshes/servo_lfs_1.stl" scale="0.001 0.001 0.001"/>
     </geometry>
   </collision>
@@ -303,5 +334,5 @@
     <origin xyz="0.059645 -0.036 -0.017875" rpy="0 0 0"/>
     <geometry>
-      <mesh filename="package://clyde_description/src/meshes/servo_lrs__1.stl" scale="0.001 0.001 0.001"/>
+      <mesh filename="file://$(find clyde_description)/src/models/clyde_model/meshes/servo_lrs__1.stl" scale="0.001 0.001 0.001"/>
     </geometry>
     <material name="silver"/>
@@ -310,125 +341,5 @@
     <origin xyz="0.059645 -0.036 -0.017875" rpy="0 0 0"/>
     <geometry>
-      <mesh filename="package://clyde_description/src/meshes/servo_lrs__1.stl" scale="0.001 0.001 0.001"/>
-    </geometry>
-  </collision>
-</link>
-<link name="a_1">
-  <inertial>
-    <origin xyz="0.0011980267759206685 0.00010035438122205087 -0.0010926527391464588" rpy="0 0 0"/>
-    <mass value="9.845210937902234e-06"/>
-    <inertia ixx="0.0" iyy="0.0" izz="0.0" ixy="0.0" iyz="-0.0" ixz="-0.0"/>
-  </inertial>
-  <visual>
-    <origin xyz="0.006412 0.032855 -0.027034" rpy="0 0 0"/>
-    <geometry>
-      <mesh filename="package://clyde_description/src/meshes/a_1.stl" scale="0.001 0.001 0.001"/>
-    </geometry>
-    <material name="silver"/>
-  </visual>
-  <collision>
-    <origin xyz="0.006412 0.032855 -0.027034" rpy="0 0 0"/>
-    <geometry>
-      <mesh filename="package://clyde_description/src/meshes/a_1.stl" scale="0.001 0.001 0.001"/>
-    </geometry>
-  </collision>
-</link>
-<link name="b__1">
-  <inertial>
-    <origin xyz="0.0012604376192366716 9.955965670559869e-05 -0.0005822422676032835" rpy="0 0 0"/>
-    <mass value="7.636356391604399e-06"/>
-    <inertia ixx="0.0" iyy="0.0" izz="0.0" ixy="-0.0" iyz="-0.0" ixz="-0.0"/>
-  </inertial>
-  <visual>
-    <origin xyz="0.002835 0.03277 -0.025616" rpy="0 0 0"/>
-    <geometry>
-      <mesh filename="package://clyde_description/src/meshes/b__1.stl" scale="0.001 0.001 0.001"/>
-    </geometry>
-    <material name="silver"/>
-  </visual>
-  <collision>
-    <origin xyz="0.002835 0.03277 -0.025616" rpy="0 0 0"/>
-    <geometry>
-      <mesh filename="package://clyde_description/src/meshes/b__1.stl" scale="0.001 0.001 0.001"/>
-    </geometry>
-  </collision>
-</link>
-<link name="c_1">
-  <inertial>
-    <origin xyz="0.0004800725906685088 0.00010010236221810742 -0.0014636091148647126" rpy="0 0 0"/>
-    <mass value="5.729215470952315e-06"/>
-    <inertia ixx="0.0" iyy="0.0" izz="0.0" ixy="0.0" iyz="-0.0" ixz="0.0"/>
-  </inertial>
-  <visual>
-    <origin xyz="-0.000594 0.032751 -0.026875" rpy="0 0 0"/>
-    <geometry>
-      <mesh filename="package://clyde_description/src/meshes/c_1.stl" scale="0.001 0.001 0.001"/>
-    </geometry>
-    <material name="silver"/>
-  </visual>
-  <collision>
-    <origin xyz="-0.000594 0.032751 -0.026875" rpy="0 0 0"/>
-    <geometry>
-      <mesh filename="package://clyde_description/src/meshes/c_1.stl" scale="0.001 0.001 0.001"/>
-    </geometry>
-  </collision>
-</link>
-<link name="d_1">
-  <inertial>
-    <origin xyz="0.0013568994912427604 9.998382103230258e-05 -0.0006094898025702025" rpy="0 0 0"/>
-    <mass value="7.529988845478445e-06"/>
-    <inertia ixx="0.0" iyy="0.0" izz="0.0" ixy="0.0" iyz="-0.0" ixz="0.0"/>
-  </inertial>
-  <visual>
-    <origin xyz="-0.002348 0.032764 -0.025618" rpy="0 0 0"/>
-    <geometry>
-      <mesh filename="package://clyde_description/src/meshes/d_1.stl" scale="0.001 0.001 0.001"/>
-    </geometry>
-    <material name="silver"/>
-  </visual>
-  <collision>
-    <origin xyz="-0.002348 0.032764 -0.025618" rpy="0 0 0"/>
-    <geometry>
-      <mesh filename="package://clyde_description/src/meshes/d_1.stl" scale="0.001 0.001 0.001"/>
-    </geometry>
-  </collision>
-</link>
-<link name="e_1">
-  <inertial>
-    <origin xyz="0.00036682874729430416 0.00010009700467959737 -0.0010508795807335665" rpy="0 0 0"/>
-    <mass value="3.2406127639379744e-06"/>
-    <inertia ixx="0.0" iyy="0.0" izz="0.0" ixy="-0.0" iyz="-0.0" ixz="0.0"/>
-  </inertial>
-  <visual>
-    <origin xyz="-0.005742 0.032834 -0.026061" rpy="0 0 0"/>
-    <geometry>
-      <mesh filename="package://clyde_description/src/meshes/e_1.stl" scale="0.001 0.001 0.001"/>
-    </geometry>
-    <material name="silver"/>
-  </visual>
-  <collision>
-    <origin xyz="-0.005742 0.032834 -0.026061" rpy="0 0 0"/>
-    <geometry>
-      <mesh filename="package://clyde_description/src/meshes/e_1.stl" scale="0.001 0.001 0.001"/>
-    </geometry>
-  </collision>
-</link>
-<link name="f_1">
-  <inertial>
-    <origin xyz="0.00026038442460935094 9.992572222918689e-05 0.00026359871408457997" rpy="0 0 0"/>
-    <mass value="6.566767036300841e-07"/>
-    <inertia ixx="0.0" iyy="0.0" izz="0.0" ixy="0.0" iyz="0.0" ixz="-0.0"/>
-  </inertial>
-  <visual>
-    <origin xyz="-0.00585 0.032837 -0.026934" rpy="0 0 0"/>
-    <geometry>
-      <mesh filename="package://clyde_description/src/meshes/f_1.stl" scale="0.001 0.001 0.001"/>
-    </geometry>
-    <material name="silver"/>
-  </visual>
-  <collision>
-    <origin xyz="-0.00585 0.032837 -0.026934" rpy="0 0 0"/>
-    <geometry>
-      <mesh filename="package://clyde_description/src/meshes/f_1.stl" scale="0.001 0.001 0.001"/>
+      <mesh filename="file://$(find clyde_description)/src/models/clyde_model/meshes/servo_lrs__1.stl" scale="0.001 0.001 0.001"/>
     </geometry>
   </collision>
@@ -443,5 +354,5 @@
     <origin xyz="-0.0525 0.0485 -0.022" rpy="0 0 0"/>
     <geometry>
-      <mesh filename="package://clyde_description/src/meshes/c_thrf__1.stl" scale="0.001 0.001 0.001"/>
+      <mesh filename="file://$(find clyde_description)/src/models/clyde_model/meshes/c_thrf__1.stl" scale="0.001 0.001 0.001"/>
     </geometry>
     <material name="silver"/>
@@ -450,125 +361,5 @@
     <origin xyz="-0.0525 0.0485 -0.022" rpy="0 0 0"/>
     <geometry>
-      <mesh filename="package://clyde_description/src/meshes/c_thrf__1.stl" scale="0.001 0.001 0.001"/>
-    </geometry>
-  </collision>
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