Commit message: settting default position as standing

File: src/clyde_description/src/urdf/clyde.urdf (robot description, URDF)
Before this commit: robot clyde, 45 links, 44 joints
Joints:
- joint shlfs_joint: origin xyz=-0.007145 0.0125 0.004125 rpy=0 0 0 -> xyz=-0.007145 0.0125 0.004125 rpy=0 -0.804 0
- joint shlft_joint: origin xyz=0.0 -0.007857 0.0 rpy=0 0 0 -> xyz=0.0 -0.007857 0.0 rpy=3.1416 1.287 3.1416
- joint shlrs_joint: origin xyz=0.007145 0.0125 0.004125 rpy=0 0 0 -> xyz=0.007145 0.0125 0.004125 rpy=0 -0.804 0
- joint shlrt_joint: origin xyz=0.0 -0.007857 0.0 rpy=0 0 0 -> xyz=0.0 -0.007857 0.0 rpy=3.1416 1.287 3.1416
- joint shrfs_joint: origin xyz=-0.007145 -0.0125 0.004125 rpy=0 0 0 -> xyz=-0.007145 -0.0125 0.004125 rpy=0 -0.804 0
- joint shrft_joint: origin xyz=0.0 0.007857 0.0 rpy=0 0 0 -> xyz=0.0 0.007857 0.0 rpy=3.1416 1.287 3.1416
- joint shrrs_joint: origin xyz=0.007145 -0.0125 0.004125 rpy=0 0 0 -> xyz=0.007145 -0.0125 0.004125 rpy=0 -0.804 0
- joint shrrt_joint: origin xyz=0.0 0.007857 0.0 rpy=0 0 0 -> xyz=0.0 0.007857 0.0 rpy=3.1416 1.287 3.1416

File: src/clyde_description/src/urdf/clyde.xacro (robot description, xacro)
@@ -878,222 +878,222 @@
   <xacro:box_inertia m="0.1" w="0.01" d="0.01" h="0.01"/>
 </link>
-<joint name="base_joint" type="fixed">
-  <parent link="base_footprint"/>
-  <child link="base_link"/>
-  <origin xyz="0.0 0.0 0.0" rpy="0 0 0"/>
-</joint>
-<joint name="Rigid 1" type="fixed">
-  <origin xyz="0.061733 -0.028 0.025792" rpy="0 0 0"/>
-  <parent link="base_link"/>
-  <child link="front__1"/>
-</joint>
-<joint name="Rigid 2" type="fixed">
-  <origin xyz="-0.061733 0.028 0.025792" rpy="0 0 0"/>
-  <parent link="base_link"/>
-  <child link="rear__1"/>
-</joint>
-<joint name="Rigid 3" type="fixed">
-  <origin xyz="0.059645 -0.036 0.017875" rpy="0 0 0"/>
-  <parent link="base_link"/>
-  <child link="servo_rfs_1"/>
-</joint>
-<joint name="Rigid 5" type="fixed">
-  <origin xyz="-0.059645 -0.036 0.017875" rpy="0 0 0"/>
-  <parent link="base_link"/>
-  <child link="servo_rrs__1"/>
-</joint>
-<joint name="Rigid 7" type="fixed">
-  <origin xyz="0.044904 0.0 0.031351" rpy="0 0 0"/>
-  <parent link="base_link"/>
-  <child link="c_neck__1"/>
-</joint>
-<joint name="Rigid 8" type="fixed">
-  <origin xyz="-0.008739 -0.00423 0.0263" rpy="0 0 0"/>
-  <parent link="jaw_1"/>
-  <child link="head__1"/>
-</joint>
-<joint name="Rigid 9" type="fixed">
-  <origin xyz="0.016896 -0.012925 -0.001914" rpy="0 0 0"/>
-  <parent link="servo_neck__1"/>
-  <child link="jaw_1"/>
-</joint>
-<joint name="Rigid 10" type="fixed">
-  <origin xyz="-0.013523 0.000445 -0.003623" rpy="0 0 0"/>
-  <parent link="th_rf_1"/>
-  <child link="tho_rf__1"/>
-</joint>
-<joint name="neck_joint" type="continuous">
-  <origin xyz="0.00265 0.0 0.00459" rpy="0.32814212668464987 -0.10093359552132034 0.5922309969483743"/>
-  <parent link="c_neck__1"/>
-  <child link="servo_neck__1"/>
-  <axis xyz="-0.5 -0.0 -0.866025"/>
-</joint>
-<joint name="Rigid 12" type="fixed">
-  <origin xyz="-0.02335 -0.001807 -0.00172" rpy="0 0 0"/>
-  <parent link="th_rf_1"/>
-  <child link="tube__1"/>
-</joint>
-<joint name="Rigid 13" type="fixed">
-  <origin xyz="0.0 -0.0023 0.0" rpy="0 0 0"/>
-  <parent link="c_thrf__1"/>
-  <child link="th_rf_1"/>
-</joint>
-<joint name="Rigid 14" type="fixed">
-  <origin xyz="-0.03091 -0.004582 -0.008283" rpy="0 0 0"/>
-  <parent link="tho_rf__1"/>
-  <child link="c_thorf_1"/>
-</joint>
-<joint name="Rigid 4" type="fixed">
-  <origin xyz="0.059645 0.036 0.017875" rpy="0 0 0"/>
-  <parent link="base_link"/>
-  <child link="servo_lfs_1"/>
-</joint>
-<joint name="Rigid 6" type="fixed">
-  <origin xyz="-0.059645 0.036 0.017875" rpy="0 0 0"/>
-  <parent link="base_link"/>
-  <child link="servo_lrs__1"/>
-</joint>
-<joint name="shrfs_joint" type="continuous">
-  <origin xyz="-0.007145 -0.0125 0.004125" rpy="0 0 0"/>
-  <parent link="servo_rfs_1"/>
-  <child link="c_thrf__1"/>
-  <axis xyz="0.0 1.0 -0.0"/>
-</joint>
-<joint name="Rigid 30" type="fixed">
-  <origin xyz="-0.008218 0.0075 0.000719" rpy="0 0 0"/>
-  <parent link="servos_rf_1"/>
-  <child link="shank_rf_1"/>
-</joint>
-<joint name="shrft_joint" type="continuous">
-  <origin xyz="0.0 0.007857 0.0" rpy="0 0 0"/>
-  <parent link="c_thorf_1"/>
-  <child link="servos_rf_1"/>
-  <axis xyz="0.0 1.0 -0.0"/>
-</joint>
-<joint name="Rigid 32" type="fixed">
-  <origin xyz="-0.013523 0.000445 -0.003623" rpy="0 0 0"/>
-  <parent link="th_rr_1"/>
-  <child link="tho_rr_1"/>
-</joint>
-<joint name="Rigid 33" type="fixed">
-  <origin xyz="-0.02335 -0.001807 -0.00172" rpy="0 0 0"/>
-  <parent link="th_rr_1"/>
-  <child link="tube_rr_1"/>
-</joint>
-<joint name="Rigid 34" type="fixed">
-  <origin xyz="0.0 -0.0023 0.0" rpy="0 0 0"/>
-  <parent link="c_thrr_1"/>
-  <child link="th_rr_1"/>
-</joint>
-<joint name="Rigid 35" type="fixed">
-  <origin xyz="-0.03091 -0.004582 -0.008283" rpy="0 0 0"/>
-  <parent link="tho_rr_1"/>
-  <child link="c_thorr_1"/>
-</joint>
-<joint name="Rigid 36" type="fixed">
-  <origin xyz="-0.008218 0.0075 0.000719" rpy="0 0 0"/>
-  <parent link="servos_rr_1"/>
-  <child link="shank_rr_1"/>
-</joint>
-<joint name="shrrs_joint" type="continuous">
-  <origin xyz="0.007145 -0.0125 0.004125" rpy="0 0 0"/>
-  <parent link="servo_rrs__1"/>
-  <child link="c_thrr_1"/>
-  <axis xyz="0.0 -1.0 -0.0"/>
-</joint>
-<joint name="shrrt_joint" type="continuous">
-  <origin xyz="0.0 0.007857 0.0" rpy="0 0 0"/>
-  <parent link="c_thorr_1"/>
-  <child link="servos_rr_1"/>
-  <axis xyz="0.0 1.0 -0.0"/>
-</joint>
-<joint name="Rigid 39" type="fixed">
-  <origin xyz="-0.013523 -0.000445 -0.003623" rpy="0 0 0"/>
-  <parent link="th_lf_1"/>
-  <child link="tho_lf_1"/>
-</joint>
-<joint name="Rigid 40" type="fixed">
-  <origin xyz="-0.02335 0.001807 -0.00172" rpy="0 0 0"/>
-  <parent link="th_lf_1"/>
-  <child link="tube_lf_1"/>
-</joint>
-<joint name="Rigid 41" type="fixed">
-  <origin xyz="0.0 0.0023 0.0" rpy="0 0 0"/>
-  <parent link="c_thlf_1"/>
-  <child link="th_lf_1"/>
-</joint>
-<joint name="Rigid 42" type="fixed">
-  <origin xyz="-0.03091 0.004582 -0.008283" rpy="0 0 0"/>
-  <parent link="tho_lf_1"/>
-  <child link="c_tholf_1"/>
-</joint>
-<joint name="Rigid 43" type="fixed">
-  <origin xyz="-0.008218 -0.007498 0.000719" rpy="0 0 0"/>
-  <parent link="servos_lf_1"/>
-  <child link="shank_lf_1"/>
-</joint>
-<joint name="shlfs_joint" type="continuous">
-  <origin xyz="-0.007145 0.0125 0.004125" rpy="0 0 0"/>
-  <parent link="servo_lfs_1"/>
-  <child link="c_thlf_1"/>
-  <axis xyz="-0.0 1.0 0.0"/>
-</joint>
-<joint name="shlft_joint" type="continuous">
-  <origin xyz="0.0 -0.007857 0.0" rpy="0 0 0"/>
-  <parent link="c_tholf_1"/>
-  <child link="servos_lf_1"/>
-  <axis xyz="-0.0 1.0 0.0"/>
-</joint>
-<joint name="Rigid 46" type="fixed">
-  <origin xyz="-0.013523 -0.000445 -0.003623" rpy="0 0 0"/>
-  <parent link="th_lr__1"/>
-  <child link="tho_lr_1"/>
-</joint>
-<joint name="Rigid 47" type="fixed">
-  <origin xyz="-0.02335 0.001807 -0.00172" rpy="0 0 0"/>
-  <parent link="th_lr__1"/>
-  <child link="tube_lr_1"/>
-</joint>
-<joint name="Rigid 48" type="fixed">
-  <origin xyz="0.0 0.002302 0.0" rpy="0 0 0"/>
-  <parent link="c_thlr_1"/>
-  <child link="th_lr__1"/>
-</joint>
-<joint name="Rigid 49" type="fixed">
-  <origin xyz="-0.03091 0.004582 -0.008283" rpy="0 0 0"/>
-  <parent link="tho_lr_1"/>
-  <child link="c_tholr__1"/>
-</joint>
-<joint name="Rigid 50" type="fixed">
-  <origin xyz="-0.008218 -0.0075 0.000719" rpy="0 0 0"/>
-  <parent link="servos_lr_1"/>
-  <child link="shank_lr_1"/>
-</joint>
-<joint name="shlrs_joint" type="continuous">
-  <origin xyz="0.007145 0.0125 0.004125" rpy="0 0 0"/>
-  <parent link="servo_lrs__1"/>
-  <child link="c_thlr_1"/>
-  <axis xyz="-0.0 -1.0 0.0"/>
-</joint>
-<joint name="shlrt_joint" type="continuous">
-  <origin xyz="0.0 -0.007857 0.0" rpy="0 0 0"/>
-  <parent link="c_tholr__1"/>
-  <child link="servos_lr_1"/>
-  <axis xyz="0.0 1.0 -0.0"/>
-</joint>
-<joint name="Rigid 58" type="fixed">
-  <origin xyz="0.0 -0.031 0.030939" rpy="0 0 0"/>
-  <parent link="base_link"/>
-  <child link="cover_1"/>
-</joint>
-<joint name="Rigid 59" type="fixed">
-  <origin xyz="-0.01725 0.0 0.023892" rpy="0 0 0"/>
-  <parent link="base_link"/>
-  <child link="battery_1"/>
-</joint>
-<joint name="imu_joint" type="fixed">
-  <parent link="base_link"/>
-  <child link="imu_link"/>
-  <origin xyz="0 0 0.03"/>
-</joint>
+  <joint name="base_joint" type="fixed">
+    <parent link="base_footprint"/>
+    <child link="base_link"/>
+    <origin rpy="0 0 0" xyz="0.0 0.0 0.0"/>
+  </joint>
+  <joint name="Rigid 1" type="fixed">
+    <origin rpy="0 0 0" xyz="0.061733 -0.028 0.025792"/>
+    <parent link="base_link"/>
+    <child link="front__1"/>
+  </joint>
+  <joint name="Rigid 2" type="fixed">
+    <origin rpy="0 0 0" xyz="-0.061733 0.028 0.025792"/>
+    <parent link="base_link"/>
+    <child link="rear__1"/>
+  </joint>
+  <joint name="Rigid 3" type="fixed">
+    <origin rpy="0 0 0" xyz="0.059645 -0.036 0.017875"/>
+    <parent link="base_link"/>
+    <child link="servo_rfs_1"/>
+  </joint>
+  <joint name="Rigid 5" type="fixed">
+    <origin rpy="0 0 0" xyz="-0.059645 -0.036 0.017875"/>
+    <parent link="base_link"/>
+    <child link="servo_rrs__1"/>
+  </joint>
+  <joint name="Rigid 7" type="fixed">
+    <origin rpy="0 0 0" xyz="0.044904 0.0 0.031351"/>
+    <parent link="base_link"/>
+    <child link="c_neck__1"/>
+  </joint>
+  <joint name="Rigid 8" type="fixed">
+    <origin rpy="0 0 0" xyz="-0.008739 -0.00423 0.0263"/>
+    <parent link="jaw_1"/>
+    <child link="head__1"/>
+  </joint>
+  <joint name="Rigid 9" type="fixed">
+    <origin rpy="0 0 0" xyz="0.016896 -0.012925 -0.001914"/>
+    <parent link="servo_neck__1"/>
+    <child link="jaw_1"/>
+  </joint>
+  <joint name="Rigid 10" type="fixed">
+    <origin rpy="0 0 0" xyz="-0.013523 0.000445 -0.003623"/>
+    <parent link="th_rf_1"/>
+    <child link="tho_rf__1"/>
+  </joint>
+  <joint name="neck_joint" type="continuous">
+    <origin rpy="0.32814212668464987 -0.10093359552132034 0.5922309969483743" xyz="0.00265 0.0 0.00459"/>
+    <parent link="c_neck__1"/>
+    <child link="servo_neck__1"/>
+    <axis xyz="-0.5 -0.0 -0.866025"/>
+  </joint>
+  <joint name="Rigid 12" type="fixed">
+    <origin rpy="0 0 0" xyz="-0.02335 -0.001807 -0.00172"/>
+    <parent link="th_rf_1"/>
+    <child link="tube__1"/>
+  </joint>
+  <joint name="Rigid 13" type="fixed">
+    <origin rpy="0 0 0" xyz="0.0 -0.0023 0.0"/>
+    <parent link="c_thrf__1"/>
+    <child link="th_rf_1"/>
+  </joint>
+  <joint name="Rigid 14" type="fixed">
+    <origin rpy="0 0 0" xyz="-0.03091 -0.004582 -0.008283"/>
+    <parent link="tho_rf__1"/>
+    <child link="c_thorf_1"/>
+  </joint>
+  <joint name="Rigid 4" type="fixed">
+    <origin rpy="0 0 0" xyz="0.059645 0.036 0.017875"/>
+    <parent link="base_link"/>
+    <child link="servo_lfs_1"/>
+  </joint>
+  <joint name="Rigid 6" type="fixed">
+    <origin rpy="0 0 0" xyz="-0.059645 0.036 0.017875"/>
+    <parent link="base_link"/>
+    <child link="servo_lrs__1"/>
+  </joint>
+  <joint name="shrfs_joint" type="continuous">
+    <origin rpy="0 -0.804 0" xyz="-0.007145 -0.0125 0.004125"/>
+    <parent link="servo_rfs_1"/>
+    <child link="c_thrf__1"/>
+    <axis xyz="0.0 1.0 -0.0"/>
+  </joint>
+  <joint name="Rigid 30" type="fixed">
+    <origin rpy="0 0 0" xyz="-0.008218 0.0075 0.000719"/>
+    <parent link="servos_rf_1"/>
+    <child link="shank_rf_1"/>
+  </joint>
+  <joint name="shrft_joint" type="continuous">
+    <origin rpy="3.1416 1.287 3.1416" xyz="0.0 0.007857 0.0"/>
+    <parent link="c_thorf_1"/>
+    <child link="servos_rf_1"/>
+    <axis xyz="0.0 1.0 -0.0"/>
+  </joint>
+  <joint name="Rigid 32" type="fixed">
+    <origin rpy="0 0 0" xyz="-0.013523 0.000445 -0.003623"/>
+    <parent link="th_rr_1"/>
+    <child link="tho_rr_1"/>
+  </joint>
+  <joint name="Rigid 33" type="fixed">
+    <origin rpy="0 0 0" xyz="-0.02335 -0.001807 -0.00172"/>
+    <parent link="th_rr_1"/>
+    <child link="tube_rr_1"/>
+  </joint>
+  <joint name="Rigid 34" type="fixed">
+    <origin rpy="0 0 0" xyz="0.0 -0.0023 0.0"/>
+    <parent link="c_thrr_1"/>
+    <child link="th_rr_1"/>
+  </joint>
+  <joint name="Rigid 35" type="fixed">
+    <origin rpy="0 0 0" xyz="-0.03091 -0.004582 -0.008283"/>
+    <parent link="tho_rr_1"/>
+    <child link="c_thorr_1"/>
+  </joint>
+  <joint name="Rigid 36" type="fixed">
+    <origin rpy="0 0 0" xyz="-0.008218 0.0075 0.000719"/>
+    <parent link="servos_rr_1"/>
+    <child link="shank_rr_1"/>
+  </joint>
+  <joint name="shrrs_joint" type="continuous">
+    <origin rpy="0 -0.804 0" xyz="0.007145 -0.0125 0.004125"/>
+    <parent link="servo_rrs__1"/>
+    <child link="c_thrr_1"/>
+    <axis xyz="0.0 -1.0 -0.0"/>
+  </joint>
+  <joint name="shrrt_joint" type="continuous">
+    <origin rpy="3.1416 1.287 3.1416" xyz="0.0 0.007857 0.0"/>
+    <parent link="c_thorr_1"/>
+    <child link="servos_rr_1"/>
+    <axis xyz="0.0 1.0 -0.0"/>
+  </joint>
+  <joint name="Rigid 39" type="fixed">
+    <origin rpy="0 0 0" xyz="-0.013523 -0.000445 -0.003623"/>
+    <parent link="th_lf_1"/>
+    <child link="tho_lf_1"/>
+  </joint>
+  <joint name="Rigid 40" type="fixed">
+    <origin rpy="0 0 0" xyz="-0.02335 0.001807 -0.00172"/>
+    <parent link="th_lf_1"/>
+    <child link="tube_lf_1"/>
+  </joint>
+  <joint name="Rigid 41" type="fixed">
+    <origin rpy="0 0 0" xyz="0.0 0.0023 0.0"/>
+    <parent link="c_thlf_1"/>
+    <child link="th_lf_1"/>
+  </joint>
+  <joint name="Rigid 42" type="fixed">
+    <origin rpy="0 0 0" xyz="-0.03091 0.004582 -0.008283"/>
+    <parent link="tho_lf_1"/>
+    <child link="c_tholf_1"/>
+  </joint>
+  <joint name="Rigid 43" type="fixed">
+    <origin rpy="0 0 0" xyz="-0.008218 -0.007498 0.000719"/>
+    <parent link="servos_lf_1"/>
+    <child link="shank_lf_1"/>
+  </joint>
+  <joint name="shlfs_joint" type="continuous">
+    <origin rpy="0 -0.804 0" xyz="-0.007145 0.0125 0.004125"/>
+    <parent link="servo_lfs_1"/>
+    <child link="c_thlf_1"/>
+    <axis xyz="-0.0 1.0 0.0"/>
+  </joint>
+  <joint name="shlft_joint" type="continuous">
+    <origin rpy="3.1416 1.287 3.1416" xyz="0.0 -0.007857 0.0"/>
+    <parent link="c_tholf_1"/>
+    <child link="servos_lf_1"/>
+    <axis xyz="-0.0 1.0 0.0"/>
+  </joint>
+  <joint name="Rigid 46" type="fixed">
+    <origin rpy="0 0 0" xyz="-0.013523 -0.000445 -0.003623"/>
+    <parent link="th_lr__1"/>
+    <child link="tho_lr_1"/>
+  </joint>
+  <joint name="Rigid 47" type="fixed">
+    <origin rpy="0 0 0" xyz="-0.02335 0.001807 -0.00172"/>
+    <parent link="th_lr__1"/>
+    <child link="tube_lr_1"/>
+  </joint>
+  <joint name="Rigid 48" type="fixed">
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
Commit message: additional joint changes

File: src/clyde_description/src/urdf/clyde.urdf (robot description, URDF)
Before this commit: robot clyde, 45 links, 44 joints
Joints:
- joint shrfs_joint: origin xyz=-0.007145 -0.0125 0.004125 rpy=0 -0.804 0 -> xyz=-0.007145 -0.0125 0.004125 rpy=0 0 0
- joint shrft_joint: origin xyz=0.0 0.007857 0.0 rpy=3.1416 1.287 3.1416 -> xyz=0.0 0.007857 0.0 rpy=0 0 0
- joint shrrs_joint: origin xyz=0.007145 -0.0125 0.004125 rpy=0 -0.804 0 -> xyz=0.007145 -0.0125 0.004125 rpy=0 0 0

File: src/clyde_description/src/urdf/clyde.xacro (robot description, xacro)
@@ -868,13 +868,13 @@
   <visual>
     <geometry>
-      <box size="0.01 0.01 0.01"/>
-    </geometry>
-  </visual>
-  <collision>
-    <geometry>
-      <box size="0.01 0.01 0.01"/>
-    </geometry>
-  </collision>
-  <xacro:box_inertia m="0.1" w="0.01" d="0.01" h="0.01"/>
+      <box size="0.02 0.02 0.004"/>
+    </geometry>
+  </visual>
+  <collision>
+    <geometry>
+      <box size="0.02 0.02 0.004"/>
+    </geometry>
+  </collision>
+  <xacro:box_inertia m="0.005" w="0.02" d="0.004" h="0.02"/>
 </link>
   <joint name="base_joint" type="fixed">
@@ -955,5 +955,5 @@
   </joint>
   <joint name="shrfs_joint" type="continuous">
-    <origin rpy="0 -0.804 0" xyz="-0.007145 -0.0125 0.004125"/>
+    <origin rpy="0 -1.375 0" xyz="-0.007145 -0.0125 0.004125"/>
     <parent link="servo_rfs_1"/>
     <child link="c_thrf__1"/>
@@ -966,5 +966,5 @@
   </joint>
   <joint name="shrft_joint" type="continuous">
-    <origin rpy="3.1416 1.287 3.1416" xyz="0.0 0.007857 0.0"/>
+    <origin rpy="0 1.240 0" xyz="0.0 0.007857 0.0"/>
     <parent link="c_thorf_1"/>
     <child link="servos_rf_1"/>
@@ -997,5 +997,5 @@
   </joint>
   <joint name="shrrs_joint" type="continuous">
-    <origin rpy="0 -0.804 0" xyz="0.007145 -0.0125 0.004125"/>
+    <origin rpy="0 -1.375 0" xyz="0.007145 -0.0125 0.004125"/>
     <parent link="servo_rrs__1"/>
     <child link="c_thrr_1"/>
@@ -1003,5 +1003,5 @@
   </joint>
   <joint name="shrrt_joint" type="continuous">
-    <origin rpy="3.1416 1.287 3.1416" xyz="0.0 0.007857 0.0"/>
+    <origin rpy="0 1.240 0" xyz="0.0 0.007857 0.0"/>
     <parent link="c_thorr_1"/>
     <child link="servos_rr_1"/>
@@ -1034,5 +1034,5 @@
   </joint>
   <joint name="shlfs_joint" type="continuous">
-    <origin rpy="0 -0.804 0" xyz="-0.007145 0.0125 0.004125"/>
+    <origin rpy="0 -1.375 0" xyz="-0.007145 0.0125 0.004125"/>
     <parent link="servo_lfs_1"/>
     <child link="c_thlf_1"/>
@@ -1040,5 +1040,5 @@
   </joint>
   <joint name="shlft_joint" type="continuous">
-    <origin rpy="3.1416 1.287 3.1416" xyz="0.0 -0.007857 0.0"/>
+    <origin rpy="0 1.240 0" xyz="0.0 -0.007857 0.0"/>
     <parent link="c_tholf_1"/>
     <child link="servos_lf_1"/>
@@ -1071,5 +1071,5 @@
   </joint>
   <joint name="shlrs_joint" type="continuous">
-    <origin rpy="0 -0.804 0" xyz="0.007145 0.0125 0.004125"/>
+    <origin rpy="0 -1.375 0" xyz="0.007145 0.0125 0.004125"/>
     <parent link="servo_lrs__1"/>
     <child link="c_thlr_1"/>
@@ -1077,5 +1077,5 @@
   </joint>
   <joint name="shlrt_joint" type="continuous">
-    <origin rpy="3.1416 1.287 3.1416" xyz="0.0 -0.007857 0.0"/>
+    <origin rpy="0 1.240 0" xyz="0.0 -0.007857 0.0"/>
     <parent link="c_tholr__1"/>
     <child link="servos_lr_1"/>

Commit message: changing default position in urdf

File: src/clyde_description/src/urdf/clyde.urdf (robot description, URDF)
Before this commit: robot clyde, 45 links, 44 joints
Links:
- link imu_link: mass 0.1 -> 0.005; geometry collision box size=0.02 0.02 0.004; visual box size=0.02 0.02 0.004
Joints:
- joint shlfs_joint: origin xyz=-0.007145 0.0125 0.004125 rpy=0 -0.804 0 -> xyz=-0.007145 0.0125 0.004125 rpy=0 -1.375 0
- joint shlft_joint: origin xyz=0.0 -0.007857 0.0 rpy=3.1416 1.287 3.1416 -> xyz=0.0 -0.007857 0.0 rpy=0 1.240 0
- joint shlrs_joint: origin xyz=0.007145 0.0125 0.004125 rpy=0 -0.804 0 -> xyz=0.007145 0.0125 0.004125 rpy=0 -1.375 0
- joint shlrt_joint: origin xyz=0.0 -0.007857 0.0 rpy=3.1416 1.287 3.1416 -> xyz=0.0 -0.007857 0.0 rpy=0 1.240 0
- joint shrfs_joint: origin xyz=-0.007145 -0.0125 0.004125 rpy=0 0 0 -> xyz=-0.007145 -0.0125 0.004125 rpy=0 -1.375 0
- joint shrft_joint: origin xyz=0.0 0.007857 0.0 rpy=0 0 0 -> xyz=0.0 0.007857 0.0 rpy=0 1.240 0
- joint shrrs_joint: origin xyz=0.007145 -0.0125 0.004125 rpy=0 0 0 -> xyz=0.007145 -0.0125 0.004125 rpy=0 -1.375 0
- joint shrrt_joint: origin xyz=0.0 0.007857 0.0 rpy=3.1416 1.287 3.1416 -> xyz=0.0 0.007857 0.0 rpy=0 1.240 0
